Commit message: fix pendulum to the world

File: urdf/pendulum.xacro (robot description, xacro)
@@ -14,4 +14,5 @@
   <xacro:property name="wheel_radius_m" value=".05" />
   <xacro:property name="wheel_length_m" value=".02" />
+  <link name="world" />
   <link name="base_link">
     <visual>
@@ -43,4 +44,8 @@
                   mass="${wheel_mass_kg}"
                   motor_mass="${motor_mass_kg}"/>
+  <joint name="fixed" type="fixed">
+    <parent link="world"/>
+    <child link="base_link"/>
+  </joint>
   <!-- Add ROS plugin so we can interact with our robot -->
   <gazebo>

Commit message: Reorient in midair to land along footfall axis
Calculate the landing angle and change the position setpoint to it.
Also debounce the contact messages. Just like real life!

Code is a little ad-hoc and messy, sorry! Needs to be cleaned up a bit.

File: urdf/pendulum.xacro (robot description, xacro)
@@ -22,5 +22,5 @@
       </geometry>
     </visual>
-    <collision>
+    <collision name="base_collision">
       <origin rpy="0 ${3.1415/2} 0" />
       <geometry>
@@ -45,4 +45,10 @@
                izz="1"/> <!-- ${base_mass_kg/12*(base_x_m**2 + base_z_m**2)} -->
     </inertial>
+    <!-- <sensor name="base_contact" type="contact">
+      <contact>
+        <collision>base_collision</collision>
+      </contact>
+      <update_rate>60</update_rate>
+    </sensor> -->
   </link>
   <xacro:arm length="${arm_length_m}"
@@ -66,5 +72,5 @@
     <plugin name="v_naught" filename="libInitialVelocityPlugin.so">
       <link>base_link</link>
-      <linear>0 0 -3.0</linear>
+      <linear>0 4.0 0</linear>
     </plugin>
   </gazebo>

Commit message: Hotfix the friction on the base link
Asking for @lkunelk 's help debugging the friction in Gazebo. It refuses
to read both the in-<link> and <gazebo> friction definitions for me, +
the CFM definition for the link.

File: urdf/pendulum.xacro (robot description, xacro)
@@ -26,4 +26,10 @@
     </inertial>
   </link> -->
+  <gazebo reference="base_link">
+    <mu1>0.2</mu1>
+    <mu2>0.2</mu2>
+    <kp>300</kp>
+    <material>Gazebo/Red</material>
+  </gazebo>
   <link name="base_link">
     <visual>
@@ -39,4 +45,9 @@
       </geometry>
       <surface>
+        <contact>
+          <ode>
+            <soft_cfm>0.3</soft_cfm>
+          </ode>
+        </contact>
         <friction>
           <ode>

Commit message: Remove name from base link collision
Friction (and kp) was being stripped from base_link during parsing because
of a bug in gazebo's URDF->SDF conversion. See osrf/gazebo#2497 . Fixing the
base link friction should eliminate the need for CFM/KP which was initially
put in to improve the collision detection with the world and stop the
robot from slipping during the pushoff phase.

File: urdf/pendulum.xacro (robot description, xacro)
@@ -27,7 +27,7 @@
   </link> -->
   <gazebo reference="base_link">
-    <mu1>0.2</mu1>
-    <mu2>0.2</mu2>
-    <kp>300</kp>
+    <mu1>200</mu1>
+    <mu2>200</mu2>
+    <!-- <kp>30000</kp> -->
     <material>Gazebo/Red</material>
   </gazebo>
@@ -39,10 +39,10 @@
       </geometry>
     </visual>
-    <collision name="base_collision">
+    <collision>
       <!-- <origin rpy="0 ${3.1415/2} 0" /> -->
       <geometry>
         <box size="0.05 0.05 0.01" />
       </geometry>
-      <surface>
+      <!-- <surface>
         <contact>
           <ode>
@@ -52,9 +52,9 @@
         <friction>
           <ode>
-            <mu>200.0</mu>
-            <mu2>200.0</mu2>
+            <mu>200</mu>
+            <mu2>200</mu2>
           </ode>
         </friction>
-      </surface>
+      </surface> -->
     </collision>
     <inertial>
