Commit message: implement PI controller - pendulum goes upright!

File: urdf/flywheel.xacro (robot description, xacro)
@@ -35,5 +35,5 @@
       </actuator>
       <joint name="arm_to_flywheel">
-        <hardwareInterface>hardware_interface/VelocityJointInterface</hardwareInterface>
+        <hardwareInterface>hardware_interface/EffortJointInterface</hardwareInterface>
       </joint>
     </transmission>

File: urdf/pendulum.xacro (robot description, xacro)
@@ -47,4 +47,5 @@
     <parent link="world"/>
     <child link="base_link"/>
+    <origin rpy="0 0 0" xyz="0 0 ${2 * base_z_m - 1}"/>
   </joint>
   <!-- Add ROS plugin so we can interact with our robot -->

Commit message: Make all principal inertias non-zero
Turns out Gazebo just really doesn't like it when the inertias are
zero. I wanted them that way so the dummy links I'm putting in to,
say, join a revolute and prismatic joint together don't affect the
simulation results. However, turns out setting them to zero does
the exact opposite and ruins the entire sim. In the first case a
few commits ago, the zero inertia on the base link was preventing
the whole robot from rotating when it hit the ground, which
happened to be fixed by adding a fixed joint to a dummy link
before the prismatic spring joint. I had thought it was a problem
with the revolute+prismatic combo somehow, but it recurred here
when adding the solenoid's prismatic joint. Now I can get rid of
all the random links that exist to put the fixed joints that
happened to stabilize the sim before. Gazebo/ODE should really be
the one here to tell you that zero inertias will pulverize your
simulation. I could understand if the result was as described in
https://wiki.ros.org/urdf/Tutorials/Adding%20Physical%20and%20Collision%20Properties%20to%20a%20URDF%20Model:

> When using realtime controllers, inertia elements of zero (or
almost zero) can cause the robot model to collapse without warning,
and all links will appear with their origins coinciding with the
world origin.

But instead we saw a robot that acted like it had infinite inertia
which is the absolute opposite of what you would expect. I had to
reconstruct the entire robot link-by-link in a separate simulation
to find this out by the way. Don't be deceived by the miniscule
changes. This was not fun.

File: urdf/flywheel.xacro (robot description, xacro)
@@ -27,5 +27,5 @@
         <origin rpy="0 0 0" xyz="0 0 0"/>
         <mass value="0.10206"/>
-        <inertia ixx="0"
+        <inertia ixx="0.000001"
                  ixy="0.00"
                  ixz="0.00"
@@ -39,5 +39,5 @@
         <origin rpy="0 0 0" xyz="0 0 0"/>
         <mass value="0.001"/>
-        <inertia ixx="0"
+        <inertia ixx="0.000001"
                  ixy="0.00"
                  ixz="0.00"
@@ -51,5 +51,5 @@
         <origin rpy="0 0 0" xyz="0 0 0"/>
         <mass value="0.001"/>
-        <inertia ixx="0"
+        <inertia ixx="0.000001"
                  ixy="0.00"
                  ixz="0.00"

File: urdf/pendulum.xacro (robot description, xacro)
@@ -37,5 +37,5 @@
     <inertial>
       <mass value="${base_mass_kg}"/>
-      <inertia ixx="0"
+      <inertia ixx="0.00000001"
                ixy="0.00"
                ixz="0.00"

Commit message: Add global constraints to robot
Force the robot into the YZ plane to reduce the instabilities of landing
on a corner of the base link. Does this defeat the purpose of using
a 3D simulator? Temporarily, yes. These are training wheels, since the
energy of the solenoid is just enough to overcome the losses baked into
the system. Note that these joints also seem to take energy out of the
system, so the simulation as a whole needs some evaluation from an
energetic standpoint.

File: urdf/flywheel.xacro (robot description, xacro)
@@ -35,35 +35,7 @@
       </inertial>
     </link>
-    <link name="arm3_link">
-      <inertial>
-        <origin rpy="0 0 0" xyz="0 0 0"/>
-        <mass value="0.001"/>
-        <inertia ixx="0.000001"
-                 ixy="0.00"
-                 ixz="0.00"
-                 iyy="0.000001"
-                 iyz="0.00"
-                 izz="0.000001"/>
-      </inertial>
-    </link>
-    <link name="arm4_link">
-      <inertial>
-        <origin rpy="0 0 0" xyz="0 0 0"/>
-        <mass value="0.001"/>
-        <inertia ixx="0.000001"
-                 ixy="0.00"
-                 ixz="0.00"
-                 iyy="0.000001"
-                 iyz="0.00"
-                 izz="0.000001"/>
-      </inertial>
-    </link>
-    <joint name="arm_arm_prism_fix" type="fixed">
-      <parent link="arm_link"/>
-      <child link="arm4_link"/>
-    </joint>
     <joint name="arm_prism" type="prismatic">
       <axis xyz="0 0 1" />
-      <parent link="arm4_link" />
+      <parent link="arm_link" />
       <child link="arm2_link" />
       <origin rpy="0 0 0" xyz="0 0 0"/>
@@ -71,11 +43,7 @@
       <limit lower="0" upper="0.013" effort="1000" velocity="1000" />
     </joint>
-    <joint name="prism_arm_fix" type="fixed">
-      <parent link="arm2_link"/>
-      <child link="arm3_link"/>
-    </joint>
     <joint name="arm_to_flywheel" type="continuous">
       <axis xyz="0 0 1"/>
-      <parent link="arm3_link"/>
+      <parent link="arm2_link"/>
       <child link="flywheel_link"/>
       <origin rpy="0 ${3.1415/2} 0" xyz="0 0 ${offset}"/>

File: urdf/pendulum.xacro (robot description, xacro)
@@ -14,4 +14,27 @@
   <xacro:property name="wheel_radius_m" value=".05" />
   <xacro:property name="wheel_length_m" value=".02" />
+  <link name="world" />
+  <link name="base0">
+    <inertial>
+      <mass value="0.0001"/>
+      <inertia ixx="0.00000001"
+               ixy="0.00"
+               ixz="0.00"
+               iyy="0.00000001"
+               iyz="0.00"
+               izz="0.00000001"/> <!-- ${base_mass_kg/12*(base_x_m**2 + base_z_m**2)} -->
+    </inertial>
+  </link>
+  <link name="base1">
+    <inertial>
+      <mass value="0.0001"/>
+      <inertia ixx="0.00000001"
+               ixy="0.00"
+               ixz="0.00"
+               iyy="0.00000001"
+               iyz="0.00"
+               izz="0.00000001"/> <!-- ${base_mass_kg/12*(base_x_m**2 + base_z_m**2)} -->
+    </inertial>
+  </link>
   <link name="base_link">
     <visual>
@@ -51,4 +74,25 @@
     </sensor> -->
   </link>
+  <joint name="world_base_theta" type="continuous">
+    <parent link="world" />
+    <child link="base0" />
+    <axis xyz="1 0 0" />
+    <origin rpy="0 0 0" xyz="0 0 0"/>
+    <limit effort="1000" velocity="1000" />
+  </joint>
+  <joint name="world_base_z" type="prismatic">
+    <parent link="base0" />
+    <child link="base1" />
+    <axis xyz="0 0 1" />
+    <origin rpy="0 0 0" xyz="0 0 0"/>
+    <limit lower="-1000" upper="1000" effort="1000" velocity="1000" />
+  </joint>
+  <joint name="world_base_y" type="prismatic">
+    <parent link="base1" />
+    <child link="base_link" />
+    <axis xyz="0 1 0" />
+    <origin rpy="0 0 0" xyz="0 0 0"/>
+    <limit lower="-1000" upper="1000" effort="1000" velocity="1000" />
+  </joint>
   <xacro:arm length="${arm_length_m}"
              width="${arm_width_m}"

Commit message: Analyze and tune solenoid
These changes are part of experiments to understand the sensitivities
of the solenoid. They revealed for the DSTL-0829 solenoid we're using
that the initial force plateau means that the energy transfer is
entirely through the speed of the body's mass, because the spring
won't compress under this force profile. This is alarming, as the
only useful part of the solenoid force is whatever it manages to
generate at maximum extension. Unfortunately, precompressing the
solenoid actually doesn't lead to significant gains even with the
optimal spring (e.g. one whose K follows the slope of the solenoid
force curve).

It's worth now exploring other options for the hopping joint.

File: urdf/flywheel.xacro (robot description, xacro)
@@ -1,5 +1,5 @@
 <?xml version="1.0"?>
 <robot xmlns:xacro="http://www.ros.org/wiki/xacro" name="pendulum">
-  <xacro:macro name="flywheel" params="radius length offset mass motor_mass">
+  <xacro:macro name="flywheel" params="radius length mass motor_mass arm_length solenoid_mass"> <!-- offset -->
     <link name="flywheel_link">
       <visual>
@@ -14,5 +14,5 @@
       </collision> -->
       <inertial>
-        <mass value="${mass + motor_mass}"/>
+        <mass value="${mass + motor_mass + solenoid_mass}"/>
         <inertia ixx="${1/12*mass*(3*radius**2 + length**2)}"
                  ixy="0.0"
@@ -26,5 +26,5 @@
       <inertial>
         <origin rpy="0 0 0" xyz="0 0 0"/>
-        <mass value="0.10206"/>
+        <mass value="0.001"/>
         <inertia ixx="0.000001"
                  ixy="0.00"
@@ -41,5 +41,5 @@
       <origin rpy="0 0 0" xyz="0 0 0"/>
       <!-- <dynamics friction="0" damping="50" /> --> <!-- implement dynamics using the PID controller (D = damping) -->
-      <limit lower="0" upper="0.013" effort="1000" velocity="1000" />
+      <limit lower="0.006" upper="0.013" effort="1000" velocity="1000" />
     </joint>
     <joint name="arm_to_flywheel" type="continuous">
@@ -47,5 +47,5 @@
       <parent link="arm2_link"/>
       <child link="flywheel_link"/>
-      <origin rpy="0 ${3.1415/2} 0" xyz="0 0 ${offset}"/>
+      <origin rpy="0 ${3.1415/2} 0" xyz="0 0 ${arm_length}"/> <!-- ${offset} -->
     </joint>
     <transmission name="$arm_prism_transmission">

File: urdf/pendulum.xacro (robot description, xacro)
@@ -12,4 +12,5 @@
   <xacro:property name="motor_mass_kg" value=".080" />
   <xacro:property name="wheel_mass_kg" value=".037" />
+  <xacro:property name="solenoid_mass_kg" value="${.10206 * 2}" />
   <xacro:property name="wheel_radius_m" value=".05" />
   <xacro:property name="wheel_length_m" value=".02" />
@@ -99,7 +100,9 @@
   <xacro:flywheel length="${wheel_length_m}"
                   radius="${wheel_radius_m}"
-                  offset="${arm_length_m}"
                   mass="${wheel_mass_kg}"
-                  motor_mass="${motor_mass_kg}"/>
+                  motor_mass="${motor_mass_kg}"
+                  arm_length="${arm_length_m}"
+                  solenoid_mass="${solenoid_mass_kg}" />
+                  <!-- offset="${arm_length_m}" -->
   <!-- <joint name="fixed" type="fixed">
     <parent link="world"/>
@@ -107,10 +110,4 @@
     <origin rpy="0 0 0" xyz="0 0 ${2 * base_z_m - 1}"/>
   </joint> -->
-  <gazebo reference="arm_link">
-    <mu1>0.2</mu1>
-    <mu2>0.2</mu2>
-    <kp>300</kp>
-    <material>Gazebo/Red</material>
-  </gazebo>
   <!-- Add ROS plugin so we can interact with our robot -->
   <gazebo>

Commit message: Shrink simulation step in the config
Needed to make the simulation resolve the servo torque limiting: it now
doesn't slam the spring into the limit, but behaves according to a
differential equation; the spring doesn't actually end up
compressing further because it's massless (see
`servo_piston_linear_analysis.ipynb` in the current `main` branch)

File: urdf/flywheel.xacro (robot description, xacro)
@@ -1,4 +1,5 @@
 <?xml version="1.0"?>
 <robot xmlns:xacro="http://www.ros.org/wiki/xacro" name="pendulum">
+  <xacro:property name="piston_offset" value="0.04" /> <!-- m -->
   <xacro:macro name="flywheel" params="radius length mass motor_mass arm_length solenoid_mass"> <!-- offset -->
     <link name="flywheel_link">
@@ -51,11 +52,11 @@
     <link name="arm3_link">
       <visual>
-        <origin rpy="0 ${3.1415/2} 0" xyz="0.01 0 0.0127"/>
+        <origin rpy="0 ${3.1415/2} 0" xyz="0.01 ${-piston_offset} 0.0"/>
         <geometry>
-          <cylinder length="0.002" radius="0.0127"/>
+          <cylinder length="0.002" radius="${piston_offset}"/>
         </geometry>
       </visual>
       <inertial>
-        <origin rpy="0 0 0" xyz="0 0 0.0127"/>
+        <origin rpy="0 0 0" xyz="0 -0.01 0.0"/>
         <mass value="0.001"/>
         <inertia ixx="0.000001"
@@ -79,4 +80,16 @@
       </inertial>
     </link>
+    <!-- <link name="arm5_link">
+      <inertial>
+        <origin rpy="0 0 0" xyz="0 0 0"/>
+        <mass value="0.001"/>
+        <inertia ixx="0.000001"
+                 ixy="0.00"
+                 ixz="0.00"
+                 iyy="0.000001"
+                 iyz="0.00"
+                 izz="0.000001"/>
+      </inertial>
+    </link> -->
     <!-- <joint name="arm_prism" type="prismatic">
       <axis xyz="0 0 1" />
@@ -102,6 +115,6 @@
       <parent link="arm3_link" />
       <child link="arm4_link" />
-      <origin rpy="0 0 0" xyz="0 0 0.0127"/>
-      <limit lower="${-3.1415*7/8}" upper="${-3.1415*1/8}" effort="1000" velocity="1000" />
+      <origin rpy="0 0 0" xyz="0 ${-piston_offset} 0"/>
+      <limit lower="0" upper="${3.1415/4}" effort="1000" velocity="1000" />
     </joint>
     <gazebo>
@@ -116,5 +129,5 @@
         <parent>arm_link</parent>
         <child>arm4_link</child>
-        <pose>0 0 0.00127 0 0 0</pose>
+        <pose>0 0 0 0 0 0</pose>
       </joint>
     </gazebo>
@@ -123,5 +136,5 @@
       <parent link="arm4_link"/>
       <child link="flywheel_link"/>
-      <origin rpy="0 ${3.1415/2} 0" xyz="0 0 ${radius}"/> <!-- ${offset} -->
+      <origin rpy="0 ${3.1415/2} 0" xyz="0 ${piston_offset} ${radius}"/> <!-- ${offset} -->
     </joint>
     <transmission name="$arm_piston_transmission">

Commit message: Ready for grid search, revert inertia values

File: urdf/flywheel.xacro (robot description, xacro)
@@ -55,5 +55,5 @@
                 <origin rpy="0 0 0" xyz="0 -0.01 0.0"/>
                 <mass value="0.001"/>
-                <inertia ixx="0.001"
+                <inertia ixx="0.000001"
                          ixy="0.00"
                          ixz="0.00"
@@ -67,5 +67,5 @@
                 <origin rpy="0 0 0" xyz="0 0 0"/>
                 <mass value="0.001"/>
-                <inertia ixx="0.001"
+                <inertia ixx="0.000001"
                          ixy="0.00"
                          ixz="0.00"
