Commit message: parametarize the pendulum

File: urdf/arm.xacro (robot description, xacro)
@@ -1,5 +1,6 @@
 <?xml version="1.0"?>
 <robot xmlns:xacro="http://www.ros.org/wiki/xacro" name="pendulum">
-<xacro:macro name="arm" params="length width">
+<xacro:macro name="arm" params="length width linear_density">
+  <xacro:property name="mass" value="${linear_density * length}" />
   <link name="arm_link">
     <visual>
@@ -17,6 +18,11 @@
     <inertial>
       <origin rpy="0 0 0" xyz="0 0 ${length/2}"/>
-      <mass value="1"/>
-      <inertia ixx="0.21" ixy="0.00" ixz="0.00" iyy="0.27" iyz="0.00" izz="0.10"/>
+      <mass value="${linear_density * length}"/>
+      <inertia ixx="${mass/12*(width**2 + width**2)}"
+               ixy="0.00"
+               ixz="0.00"
+               iyy="${mass/12*(width**2 + width**2)}"
+               iyz="0.00"
+               izz="${mass/12*(width**2 + width**2)}"/>
     </inertial>
   </link>
@@ -27,5 +33,4 @@
     <origin rpy="0 0 0" xyz="0 0 0"/>
   </joint>
-  <xacro:flywheel length="0.02" radius="0.05" offset="${length}" />
 </xacro:macro>
 </robot>

File: urdf/flywheel.xacro (robot description, xacro)
@@ -1,5 +1,5 @@
 <?xml version="1.0"?>
 <robot xmlns:xacro="http://www.ros.org/wiki/xacro" name="pendulum">
-  <xacro:macro name="flywheel" params="radius length offset">
+  <xacro:macro name="flywheel" params="radius length offset mass motor_mass">
     <link name="flywheel_link">
       <visual>
@@ -14,6 +14,11 @@
       </collision>
       <inertial>
-        <mass value="1"/>
-        <inertia ixx="0.06" ixy="0.0" ixz="0.0" iyy="0.06" iyz="0.0" izz="0.25"/>
+        <mass value="${mass + motor_mass}"/>
+        <inertia ixx="${1/12*mass*(3*radius**2 + length**2)}"
+                 ixy="0.0"
+                 ixz="0.0"
+                 iyy="${1/12*mass*(3*radius**2 + length**2)}"
+                 iyz="0.0"
+                 izz="${1/2*mass*(radius**2)}"/>
       </inertial>
     </link>

File: urdf/pendulum.xacro (robot description, xacro)
@@ -3,21 +3,44 @@
   <xacro:include filename="$(find pendulum)/urdf/arm.xacro" />
   <xacro:include filename="$(find pendulum)/urdf/flywheel.xacro" />
+  <xacro:property name="base_mass_kg" value="100" />
+  <xacro:property name="base_x_m" value=".05" />
+  <xacro:property name="base_y_m" value=".05" />
+  <xacro:property name="base_z_m" value=".06" />
+  <xacro:property name="arm_linear_density_kg_m" value=".129" />
+  <xacro:property name="arm_length_m" value=".10" />
+  <xacro:property name="arm_width_m" value=".02" />
+  <xacro:property name="motor_mass_kg" value=".186" />
+  <xacro:property name="wheel_mass_kg" value=".037" />
+  <xacro:property name="wheel_radius_m" value=".05" />
+  <xacro:property name="wheel_length_m" value=".02" />
   <link name="base_link">
     <visual>
       <geometry>
-        <box size=".10 .10 .05"/>
+        <box size="${base_x_m} ${base_y_m} ${base_z_m}"/>
       </geometry>
     </visual>
     <collision>
       <geometry>
-        <box size=".10 .10 .05"/>
+        <box size="${base_x_m} ${base_y_m} ${base_z_m}"/>
       </geometry>
     </collision>
     <inertial>
-      <mass value="100"/>
-      <inertia ixx="10.0" ixy="0.00" ixz="0.00" iyy="10.0" iyz="0.00" izz="10.0"/>
+      <mass value="${base_mass_kg}"/>
+      <inertia ixx="${base_mass_kg/12*(base_y_m**2 + base_z_m**2)}"
+               ixy="0.00"
+               ixz="0.00"
+               iyy="${base_mass_kg/12*(base_x_m**2 + base_z_m**2)}"
+               iyz="0.00"
+               izz="${base_mass_kg/12*(base_x_m**2 + base_y_m**2)}"/>
     </inertial>
   </link>
-  <xacro:arm length="0.30" width="0.02" />
+  <xacro:arm length="${arm_length_m}"
+             width="${arm_width_m}"
+             linear_density="${arm_linear_density_kg_m}"/>
+  <xacro:flywheel length="${wheel_length_m}"
+                  radius="${wheel_radius_m}"
+                  offset="${arm_length_m}"
+                  mass="${wheel_mass_kg}"
+                  motor_mass="${motor_mass_kg}"/>
   <!-- Add ROS plugin so we can interact with our robot -->
   <gazebo>

Commit message: add arm angle limit, control limits for torque and speed based on motor parameter

File: urdf/arm.xacro (robot description, xacro)
@@ -27,9 +27,10 @@
     </inertial>
   </link>
-  <joint name="base_to_arm" type="continuous">
+  <joint name="base_to_arm" type="revolute">
     <axis xyz="1 0 0"/>
     <parent link="base_link"/>
     <child link="arm_link"/>
     <origin rpy="0 0 0" xyz="0 0 0"/>
+    <limit effort="100" upper="0.5" lower="-0.5" velocity="1000"/>
   </joint>
 </xacro:macro>

File: urdf/pendulum.xacro (robot description, xacro)
@@ -10,5 +10,5 @@
   <xacro:property name="arm_length_m" value=".10" />
   <xacro:property name="arm_width_m" value=".02" />
-  <xacro:property name="motor_mass_kg" value=".186" />
+  <xacro:property name="motor_mass_kg" value=".080" />
   <xacro:property name="wheel_mass_kg" value=".037" />
   <xacro:property name="wheel_radius_m" value=".05" />

Commit message: add motor to base_arm joint

File: urdf/arm.xacro (robot description, xacro)
@@ -32,6 +32,15 @@
     <child link="arm_link"/>
     <origin rpy="0 0 0" xyz="0 0 0"/>
-    <limit effort="100" upper="0.5" lower="-0.5" velocity="1000"/>
+    <limit effort="100" upper="1.5708" lower="-1.5708" velocity="1000"/>
   </joint>
+  <transmission name="$arm_transmission">
+    <type>transmission_interface/SimpleTransmission</type>
+    <actuator name="$arm_motor">
+      <mechanicalReduction>1</mechanicalReduction>
+    </actuator>
+    <joint name="base_to_arm">
+      <hardwareInterface>hardware_interface/EffortJointInterface</hardwareInterface>
+    </joint>
+  </transmission>
 </xacro:macro>
 </robot>

Commit message: Added control for prismatic joint

File: urdf/arm.xacro (robot description, xacro)
@@ -10,10 +10,10 @@
       </geometry>
     </visual>
-    <collision>
+    <!--collision>
       <origin rpy="0 0 0" xyz="0 0 ${length/2}"/>
       <geometry>
         <box size="${width} ${width} ${length}"/>
       </geometry>
-    </collision>
+    </collision-->
     <inertial>
       <origin rpy="0 0 0" xyz="0 0 ${length/2}"/>
@@ -27,12 +27,21 @@
     </inertial>
   </link>
+  <!-- <link name="arm0_link">
+  </link>
   <joint name="base_to_arm" type="revolute">
     <axis xyz="1 0 0"/>
     <parent link="base_link"/>
-    <child link="arm_link"/>
+    <child link="arm0_link"/>
     <origin rpy="0 0 0" xyz="0 0 0"/>
     <limit effort="100" upper="1.5708" lower="-1.5708" velocity="1000"/>
+  </joint> -->
+  <joint name="arm_prism" type="prismatic">
+    <axis xyz="0 0 1" />
+    <parent link="base_link" />
+    <child link="arm_link" />
+    <origin rpy="0 0 0" xyz="0 0 0"/>
+    <limit effort="1000" velocity="1000" />
   </joint>
-  <transmission name="$arm_transmission">
+  <!-- <transmission name="$arm_transmission">
     <type>transmission_interface/SimpleTransmission</type>
     <actuator name="$arm_motor">
@@ -42,4 +51,13 @@
       <hardwareInterface>hardware_interface/EffortJointInterface</hardwareInterface>
     </joint>
+  </transmission> -->
+  <transmission name="$arm_prism_transmission">
+    <type>transmission_interface/SimpleTransmission</type>
+    <actuator name="$arm_prism_motor">
+      <mechanicalReduction>1</mechanicalReduction>
+    </actuator>
+    <joint name="arm_prism">
+      <hardwareInterface>hardware_interface/EffortJointInterface</hardwareInterface>
+    </joint>
   </transmission>
 </xacro:macro>

File: urdf/pendulum.xacro (robot description, xacro)
@@ -3,5 +3,5 @@
   <xacro:include filename="$(find pendulum)/urdf/arm.xacro" />
   <xacro:include filename="$(find pendulum)/urdf/flywheel.xacro" />
-  <xacro:property name="base_mass_kg" value="100" />
+  <xacro:property name="base_mass_kg" value="10" />
   <xacro:property name="base_x_m" value=".05" />
   <xacro:property name="base_y_m" value=".05" />
@@ -14,24 +14,34 @@
   <xacro:property name="wheel_radius_m" value=".05" />
   <xacro:property name="wheel_length_m" value=".02" />
-  <link name="world" />
+  <!-- <link name="world" /> -->
   <link name="base_link">
     <visual>
+      <origin rpy="0 ${3.1415/2} 0" />
       <geometry>
-        <box size="${base_x_m} ${base_y_m} ${base_z_m}"/>
+        <cylinder radius="0.01" length="0.05" />
       </geometry>
     </visual>
     <collision>
+      <origin rpy="0 ${3.1415/2} 0" />
       <geometry>
-        <box size="${base_x_m} ${base_y_m} ${base_z_m}"/>
+        <cylinder radius="0.01" length="0.05" />
       </geometry>
+      <surface>
+        <friction>
+          <ode>
+            <mu>10000</mu>
+            <mu2>10000</mu2>
+          </ode>
+        </friction>
+      </surface>
     </collision>
     <inertial>
       <mass value="${base_mass_kg}"/>
-      <inertia ixx="${base_mass_kg/12*(base_y_m**2 + base_z_m**2)}"
+      <inertia ixx="0.00"
                ixy="0.00"
                ixz="0.00"
-               iyy="${base_mass_kg/12*(base_x_m**2 + base_z_m**2)}"
+               iyy="10"
                iyz="0.00"
-               izz="${base_mass_kg/12*(base_x_m**2 + base_y_m**2)}"/>
+               izz="10"/> <!-- ${base_mass_kg/12*(base_x_m**2 + base_z_m**2)} -->
     </inertial>
   </link>
@@ -44,9 +54,9 @@
                   mass="${wheel_mass_kg}"
                   motor_mass="${motor_mass_kg}"/>
-  <joint name="fixed" type="fixed">
+  <!-- <joint name="fixed" type="fixed">
     <parent link="world"/>
     <child link="base_link"/>
     <origin rpy="0 0 0" xyz="0 0 ${2 * base_z_m - 1}"/>
-  </joint>
+  </joint> -->
   <!-- Add ROS plugin so we can interact with our robot -->
   <gazebo>

Commit message: Debug prismatic joint + default offset
Prismatic joint is now working with a PID controller (command emitted
by main controller which is a bit weird but works for now). Also, the
sim now starts with an initial rotation using the command-line option
in the gazebo.launch file. Both are in service of simulating the foot
fall of the robot.

File: urdf/arm.xacro (robot description, xacro)
@@ -27,19 +27,41 @@
     </inertial>
   </link>
-  <!-- <link name="arm0_link">
+  <link name="arm0_link">
+    <!-- <visual>
+      <origin rpy="0 0 0" xyz="0 0 ${length/2}"/>
+      <geometry>
+        <box size="${width} ${width} ${length}"/>
+      </geometry>
+    </visual> -->
+    <!--collision>
+      <origin rpy="0 0 0" xyz="0 0 ${length/2}"/>
+      <geometry>
+        <box size="${width} ${width} ${length}"/>
+      </geometry>
+    </collision-->
+    <inertial>
+      <origin rpy="0 0 0" xyz="0 0 ${length/2}"/>
+      <mass value="${linear_density * length}"/>
+      <inertia ixx="0"
+               ixy="0.00"
+               ixz="0.00"
+               iyy="10"
+               iyz="0.00"
+               izz="10"/>
+    </inertial>
   </link>
-  <joint name="base_to_arm" type="revolute">
+  <joint name="base_to_arm" type="continuous">
     <axis xyz="1 0 0"/>
     <parent link="base_link"/>
     <child link="arm0_link"/>
     <origin rpy="0 0 0" xyz="0 0 0"/>
-    <limit effort="100" upper="1.5708" lower="-1.5708" velocity="1000"/>
-  </joint> -->
+    <limit effort="100" velocity="1000"/>
+  </joint>
   <joint name="arm_prism" type="prismatic">
     <axis xyz="0 0 1" />
-    <parent link="base_link" />
+    <parent link="arm0_link" />
     <child link="arm_link" />
     <origin rpy="0 0 0" xyz="0 0 0"/>
-    <limit effort="1000" velocity="1000" />
+    <limit lower="-1" upper="1" effort="1000" velocity="1000" />
   </joint>
   <!-- <transmission name="$arm_transmission">

Commit message: Make a pendulum that swings on impact
Strangely, the choice of joints in the robot seems to impact what
the landing behavior is very strongly. In a separate stash (to be
committed), the robot bounces on impact, whereas here we get the
expected behavior of the arm swinging due to the momentum of the
motor and wheel.

This situation is much more challenging for the controller, which
performed confusingly well in the other scenario; now we know it's
because the momentum somehow disappears.

File: urdf/arm.xacro (robot description, xacro)
@@ -51,5 +51,5 @@
     </inertial>
   </link>
-  <joint name="base_to_arm" type="continuous">
+  <joint name="base_to_arm" type="fixed">
     <axis xyz="1 0 0"/>
     <parent link="base_link"/>

File: urdf/flywheel.xacro (robot description, xacro)
@@ -8,9 +8,9 @@
         </geometry>
       </visual>
-      <collision>
+      <!-- <collision>
         <geometry>
           <cylinder length="${length}" radius="${radius}"/>
         </geometry>
-      </collision>
+      </collision> -->
       <inertial>
         <mass value="${mass + motor_mass}"/>

File: urdf/pendulum.xacro (robot description, xacro)
@@ -3,5 +3,5 @@
   <xacro:include filename="$(find pendulum)/urdf/arm.xacro" />
   <xacro:include filename="$(find pendulum)/urdf/flywheel.xacro" />
-  <xacro:property name="base_mass_kg" value="10" />
+  <xacro:property name="base_mass_kg" value="0.01" />
   <xacro:property name="base_x_m" value=".05" />
   <xacro:property name="base_y_m" value=".05" />

Commit message: Throw it on the grouuund
Add an initial velocity so the controller doesn't have time to correct
the initial angle too much, so we know what the behavior is like when
it impacts at an angle. Also tweak the urdf params for more realistic
physics.

File: urdf/arm.xacro (robot description, xacro)
@@ -28,16 +28,4 @@
   </link>
   <link name="arm0_link">
-    <!-- <visual>
-      <origin rpy="0 0 0" xyz="0 0 ${length/2}"/>
-      <geometry>
-        <box size="${width} ${width} ${length}"/>
-      </geometry>
-    </visual> -->
-    <!--collision>
-      <origin rpy="0 0 0" xyz="0 0 ${length/2}"/>
-      <geometry>
-        <box size="${width} ${width} ${length}"/>
-      </geometry>
-    </collision-->
     <inertial>
       <origin rpy="0 0 0" xyz="0 0 ${length/2}"/>
@@ -63,4 +51,5 @@
     <child link="arm_link" />
     <origin rpy="0 0 0" xyz="0 0 0"/>
+    <!-- <dynamics friction="0" damping="50" /> --> <!-- implement dynamics using the PID controller (D = damping) -->
     <limit lower="-1" upper="1" effort="1000" velocity="1000" />
   </joint>

File: urdf/pendulum.xacro (robot description, xacro)
@@ -3,5 +3,5 @@
   <xacro:include filename="$(find pendulum)/urdf/arm.xacro" />
   <xacro:include filename="$(find pendulum)/urdf/flywheel.xacro" />
-  <xacro:property name="base_mass_kg" value="0.01" />
+  <xacro:property name="base_mass_kg" value="0.001" />
   <xacro:property name="base_x_m" value=".05" />
   <xacro:property name="base_y_m" value=".05" />
@@ -30,6 +30,6 @@
         <friction>
           <ode>
-            <mu>10000</mu>
-            <mu2>10000</mu2>
+            <mu>0.6</mu>
+            <mu2>0.6</mu2>
           </ode>
         </friction>
@@ -41,7 +41,7 @@
                ixy="0.00"
                ixz="0.00"
-               iyy="10"
+               iyy="1"
                iyz="0.00"
-               izz="10"/> <!-- ${base_mass_kg/12*(base_x_m**2 + base_z_m**2)} -->
+               izz="1"/> <!-- ${base_mass_kg/12*(base_x_m**2 + base_z_m**2)} -->
     </inertial>
   </link>
@@ -64,4 +64,8 @@
       <robotNamespace>/</robotNamespace>
     </plugin>
+    <plugin name="v_naught" filename="libInitialVelocityPlugin.so">
+      <link>base_link</link>
+      <linear>0 0 -3.0</linear>
+    </plugin>
   </gazebo>
 </robot>

Commit message: Make custom node for prismatic joint controller
Implement a custom controller for the prismatic joint, implementing the spring
within as well. This controller for now applies a constant force whenever the
joint is expanding to increase jump height over time.

Note the joint controller rate needed to be updated because the existing 50Hz
was too slow for the spring physics to converge. I don't know if we really
_need_ 1kHz but it does (seem to) work at that rate at least.

Also refactor the contact detection to its own separate node now that two
controllers are using it.

File: urdf/arm.xacro (robot description, xacro)
@@ -30,5 +30,5 @@
     <inertial>
       <origin rpy="0 0 0" xyz="0 0 ${length/2}"/>
-      <mass value="${linear_density * length}"/>
+      <mass value="0.001"/>
       <inertia ixx="0"
                ixy="0.00"
@@ -52,5 +52,5 @@
     <origin rpy="0 0 0" xyz="0 0 0"/>
     <!-- <dynamics friction="0" damping="50" /> --> <!-- implement dynamics using the PID controller (D = damping) -->
-    <limit lower="-1" upper="1" effort="1000" velocity="1000" />
+    <limit lower="-1" upper="0" effort="1000" velocity="1000" />
   </joint>
   <!-- <transmission name="$arm_transmission">

File: urdf/pendulum.xacro (robot description, xacro)
@@ -70,8 +70,8 @@
       <robotNamespace>/</robotNamespace>
     </plugin>
-    <plugin name="v_naught" filename="libInitialVelocityPlugin.so">
+    <!-- <plugin name="v_naught" filename="libInitialVelocityPlugin.so">
       <link>base_link</link>
       <linear>0 4.0 0</linear>
-    </plugin>
+    </plugin> -->
   </gazebo>
 </robot>

Commit message: Implement hopping with a pull solenoid
Pull on the solenoid as the robot lifts off the ground to compress a
spring, let go when the robot is at the bottom of its bounce. Surprisingly
the energy transfer is not very efficient and the bounce seems to get lost
in the default frictions of the system. To my understanding this is already
among the best timings for a pull solenoid.

A push solenoid transfers more energy by foregoing the energy storage spring
altogether, and of course you can make one by just flipping one of the links
around. Let's try that next.

File: urdf/arm.xacro (robot description, xacro)
@@ -29,5 +29,6 @@
   <link name="arm0_link">
     <inertial>
-      <origin rpy="0 0 0" xyz="0 0 ${length/2}"/>
+      <origin rpy="0 0 0" xyz="0 0 0"/>
+      <!-- holds the mass of the solenoid, DSTL-0829-12 -->
       <mass value="0.001"/>
       <inertia ixx="0"
@@ -39,19 +40,52 @@
     </inertial>
   </link>
+  <!-- <link name="arm1_link">
+    <inertial>
+      <origin rpy="0 0 0" xyz="0 0 0"/>
+      <mass value="0.001"/>
+      <inertia ixx="0"
+               ixy="0.00"
+               ixz="0.00"
+               iyy="10"
+               iyz="0.00"
+               izz="10"/>
+    </inertial>
+  </link> -->
+  <link name="arm2_link">
+    <inertial>
+      <origin rpy="0 0 0" xyz="0 0 0"/>
+      <mass value="0.10206"/>
+      <inertia ixx="0"
+               ixy="0.00"
+               ixz="0.00"
+               iyy="10"
+               iyz="0.00"
+               izz="10"/>
+    </inertial>
+  </link>
   <joint name="base_to_arm" type="fixed">
-    <axis xyz="1 0 0"/>
     <parent link="base_link"/>
     <child link="arm0_link"/>
-    <origin rpy="0 0 0" xyz="0 0 0"/>
-    <limit effort="100" velocity="1000"/>
   </joint>
   <joint name="arm_prism" type="prismatic">
     <axis xyz="0 0 1" />
     <parent link="arm0_link" />
+    <child link="arm2_link" />
+    <origin rpy="0 0 0" xyz="0 0 0"/>
+    <!-- <dynamics friction="0" damping="50" /> --> <!-- implement dynamics using the PID controller (D = damping) -->
+    <limit lower="-0.013" upper="0" effort="1000" velocity="1000" />
+  </joint>
+  <joint name="arm_spring" type="prismatic">
+    <axis xyz="0 0 1" />
+    <parent link="arm2_link" />
     <child link="arm_link" />
     <origin rpy="0 0 0" xyz="0 0 0"/>
     <!-- <dynamics friction="0" damping="50" /> --> <!-- implement dynamics using the PID controller (D = damping) -->
-    <limit lower="-1" upper="0" effort="1000" velocity="1000" />
+    <limit lower="-1" upper="1" effort="1000" velocity="1000" />
   </joint>
+  <!-- <joint name="arm_fix" type="fixed">
+    <parent link="arm1_link" />
+    <child link="arm2_link" />
+  </joint> -->
   <!-- <transmission name="$arm_transmission">
     <type>transmission_interface/SimpleTransmission</type>
@@ -63,4 +97,13 @@
     </joint>
   </transmission> -->
+  <transmission name="$arm_spring_transmission">
+    <type>transmission_interface/SimpleTransmission</type>
+    <actuator name="$arm_spring_motor">
+      <mechanicalReduction>1</mechanicalReduction>
+    </actuator>
+    <joint name="arm_spring">
+      <hardwareInterface>hardware_interface/EffortJointInterface</hardwareInterface>
+    </joint>
+  </transmission>
   <transmission name="$arm_prism_transmission">
     <type>transmission_interface/SimpleTransmission</type>
