Commit message: Use solenoid on push stroke, move to top of pendulum
Using a separate spring to store the solenoid energy is inefficient,
because the solenoid force is non-linear with length, so any spring
would either be too stiff near equilibrium, or too soft at max
compression. This is detailed in the previous commit too. Now, the
solenoid uses a push stroke (to be achieved physically by flipping
one of the interfaces to the links upside down and using a pull stroke)
and is able to deliver more energy.

Also, @lkunelk 's suggestion fixed the energy loss issue from the
inelastic collisions at the solenoid and spring end stops by putting
all the mass on one end, so the systems before and after the collision
don't differ much in mass and energy is mostly preserved.

File: urdf/arm.xacro (robot description, xacro)
@@ -52,35 +52,15 @@
     </inertial>
   </link> -->
-  <link name="arm2_link">
-    <inertial>
-      <origin rpy="0 0 0" xyz="0 0 0"/>
-      <mass value="0.10206"/>
-      <inertia ixx="0"
-               ixy="0.00"
-               ixz="0.00"
-               iyy="10"
-               iyz="0.00"
-               izz="10"/>
-    </inertial>
-  </link>
   <joint name="base_to_arm" type="fixed">
     <parent link="base_link"/>
     <child link="arm0_link"/>
   </joint>
-  <joint name="arm_prism" type="prismatic">
+  <joint name="arm_spring" type="prismatic">
     <axis xyz="0 0 1" />
     <parent link="arm0_link" />
-    <child link="arm2_link" />
-    <origin rpy="0 0 0" xyz="0 0 0"/>
-    <!-- <dynamics friction="0" damping="50" /> --> <!-- implement dynamics using the PID controller (D = damping) -->
-    <limit lower="-0.013" upper="0" effort="1000" velocity="1000" />
-  </joint>
-  <joint name="arm_spring" type="prismatic">
-    <axis xyz="0 0 1" />
-    <parent link="arm2_link" />
     <child link="arm_link" />
     <origin rpy="0 0 0" xyz="0 0 0"/>
     <!-- <dynamics friction="0" damping="50" /> --> <!-- implement dynamics using the PID controller (D = damping) -->
-    <limit lower="-1" upper="1" effort="1000" velocity="1000" />
+    <limit lower="-1" upper="0" effort="1000" velocity="1000" />
   </joint>
   <!-- <joint name="arm_fix" type="fixed">

File: urdf/flywheel.xacro (robot description, xacro)
@@ -23,10 +23,39 @@
       </inertial>
     </link>
+    <link name="arm2_link">
+      <inertial>
+        <origin rpy="0 0 0" xyz="0 0 0"/>
+        <mass value="0.10206"/>
+        <inertia ixx="0"
+                 ixy="0.00"
+                 ixz="0.00"
+                 iyy="10"
+                 iyz="0.00"
+                 izz="10"/>
+      </inertial>
+    </link>
+    <joint name="arm_prism" type="prismatic">
+      <axis xyz="0 0 1" />
+      <parent link="arm_link" />
+      <child link="arm2_link" />
+      <origin rpy="0 0 0" xyz="0 0 0"/>
+      <!-- <dynamics friction="0" damping="50" /> --> <!-- implement dynamics using the PID controller (D = damping) -->
+      <limit lower="0" upper="0.013" effort="1000" velocity="1000" />
+    </joint>
     <joint name="arm_to_flywheel" type="continuous">
       <axis xyz="0 0 1"/>
-      <parent link="arm_link"/>
+      <parent link="arm2_link"/>
       <child link="flywheel_link"/>
       <origin rpy="0 ${3.1415/2} 0" xyz="0 0 ${offset}"/>
     </joint>
+    <transmission name="$arm_prism_transmission">
+      <type>transmission_interface/SimpleTransmission</type>
+      <actuator name="$arm_prism_motor">
+        <mechanicalReduction>1</mechanicalReduction>
+      </actuator>
+      <joint name="arm_prism">
+        <hardwareInterface>hardware_interface/EffortJointInterface</hardwareInterface>
+      </joint>
+    </transmission>
     <transmission name="$flywheel_transmission">
       <type>transmission_interface/SimpleTransmission</type>

Commit message: Begin tracking a 1D path
Reorient while lifting off to track a position given by a tracker object
in the world. Involved some refactors because link and joint
orders
started changing based on which model was read in first.

File: urdf/arm.xacro (robot description, xacro)
@@ -35,7 +35,7 @@
                ixy="0.00"
                ixz="0.00"
-               iyy="10"
+               iyy="0.0000001"
                iyz="0.00"
-               izz="10"/>
+               izz="0.0000001"/>
     </inertial>
   </link>

File: urdf/flywheel.xacro (robot description, xacro)
@@ -30,12 +30,40 @@
                  ixy="0.00"
                  ixz="0.00"
-                 iyy="10"
+                 iyy="0.000001"
                  iyz="0.00"
-                 izz="10"/>
+                 izz="0.000001"/>
       </inertial>
     </link>
+    <link name="arm3_link">
+      <inertial>
+        <origin rpy="0 0 0" xyz="0 0 0"/>
+        <mass value="0.001"/>
+        <inertia ixx="0"
+                 ixy="0.00"
+                 ixz="0.00"
+                 iyy="0.000001"
+                 iyz="0.00"
+                 izz="0.000001"/>
+      </inertial>
+    </link>
+    <link name="arm4_link">
+      <inertial>
+        <origin rpy="0 0 0" xyz="0 0 0"/>
+        <mass value="0.001"/>
+        <inertia ixx="0"
+                 ixy="0.00"
+                 ixz="0.00"
+                 iyy="0.000001"
+                 iyz="0.00"
+                 izz="0.000001"/>
+      </inertial>
+    </link>
+    <joint name="arm_arm_prism_fix" type="fixed">
+      <parent link="arm_link"/>
+      <child link="arm4_link"/>
+    </joint>
     <joint name="arm_prism" type="prismatic">
       <axis xyz="0 0 1" />
-      <parent link="arm_link" />
+      <parent link="arm4_link" />
       <child link="arm2_link" />
       <origin rpy="0 0 0" xyz="0 0 0"/>
@@ -43,7 +71,11 @@
       <limit lower="0" upper="0.013" effort="1000" velocity="1000" />
     </joint>
+    <joint name="prism_arm_fix" type="fixed">
+      <parent link="arm2_link"/>
+      <child link="arm3_link"/>
+    </joint>
     <joint name="arm_to_flywheel" type="continuous">
       <axis xyz="0 0 1"/>
-      <parent link="arm2_link"/>
+      <parent link="arm3_link"/>
       <child link="flywheel_link"/>
       <origin rpy="0 ${3.1415/2} 0" xyz="0 0 ${offset}"/>

File: urdf/pendulum.xacro (robot description, xacro)
@@ -14,5 +14,4 @@
   <xacro:property name="wheel_radius_m" value=".05" />
   <xacro:property name="wheel_length_m" value=".02" />
-  <!-- <link name="world" /> -->
   <link name="base_link">
     <visual>
@@ -38,10 +37,10 @@
     <inertial>
       <mass value="${base_mass_kg}"/>
-      <inertia ixx="0.00"
+      <inertia ixx="0"
                ixy="0.00"
                ixz="0.00"
-               iyy="1"
+               iyy="0.00000001"
                iyz="0.00"
-               izz="1"/> <!-- ${base_mass_kg/12*(base_x_m**2 + base_z_m**2)} -->
+               izz="0.00000001"/> <!-- ${base_mass_kg/12*(base_x_m**2 + base_z_m**2)} -->
     </inertial>
     <!-- <sensor name="base_contact" type="contact">

Commit message: Better estimate landing angle, re-enable path tracking
Previously, we were using the position of the base link to estimate the
trajectory of the robot, but as the robot repositioned to land, the
link would swivel and threw off the estimate. The ideal solution is to
track the center of mass, and now that almost all the mass is at the
top of the robot, we can just track the flywheel. However, the flywheel
isn't the part that's hitting the ground, so we have to compensate.

The equations coming from conservation of energy originally made the
landing velocity very easy to calculate, but having to compensate for
the angle of the arm, which is itself dependent on the landing velocity,
makes the equation not fun analytically. Instead, it turns out that we
can just run it as a recurrence relation, because the way it is done in
`main.cpp` always overestimates the landing height and is hence stable.
In practice, it converges very quickly, to within 3 significant digits
in a couple of iterations.

Now the robot is bouncing everywhere, it's also important to refactor
the base link. To help things out a bit, this commit makes the base
link into a proper foot with a wide and short box, and gives it a very
high inertia in all axes so it stays locked to its initial world
orientation. This removes the need for the world constraint joints
which caused problems keeping the energy inside the robot before.

Housekeeping note: joint and link state message accesses are being
modified to index by searching the name in the `names` fields
instead of using fixed numeric indices. These were coming in
unreliable order, seemingly because of the addition of the tracking
dot that made a race condition for which robot was loaded first. This
commit begins util and const files to house these housekeeping items.

File: urdf/arm.xacro (robot description, xacro)
@@ -1,5 +1,5 @@
 <?xml version="1.0"?>
 <robot xmlns:xacro="http://www.ros.org/wiki/xacro" name="pendulum">
-<xacro:macro name="arm" params="length width linear_density">
+  <xacro:macro name="arm" params="length width linear_density">
   <xacro:property name="mass" value="${linear_density * length}" />
   <link name="arm_link">
@@ -32,5 +32,5 @@
       <!-- holds the mass of the solenoid, DSTL-0829-12 -->
       <mass value="0.001"/>
-      <inertia ixx="0"
+      <inertia ixx="0.0000001"
                ixy="0.00"
                ixz="0.00"
@@ -52,7 +52,10 @@
     </inertial>
   </link> -->
-  <joint name="base_to_arm" type="fixed">
-    <parent link="base_link"/>
-    <child link="arm0_link"/>
+  <joint name="base_free_theta" type="continuous">
+    <parent link="base_link" />
+    <child link="arm0_link" />
+    <axis xyz="1 0 0" />
+    <origin rpy="0 0 0" xyz="0 0 0"/>
+    <limit effort="1000" velocity="1000" />
   </joint>
   <joint name="arm_spring" type="prismatic">

File: urdf/pendulum.xacro (robot description, xacro)
@@ -14,16 +14,5 @@
   <xacro:property name="wheel_radius_m" value=".05" />
   <xacro:property name="wheel_length_m" value=".02" />
-  <link name="world" />
-  <link name="base0">
-    <inertial>
-      <mass value="0.0001"/>
-      <inertia ixx="0.00000001"
-               ixy="0.00"
-               ixz="0.00"
-               iyy="0.00000001"
-               iyz="0.00"
-               izz="0.00000001"/> <!-- ${base_mass_kg/12*(base_x_m**2 + base_z_m**2)} -->
-    </inertial>
-  </link>
+  <!-- <link name="world" />
   <link name="base1">
     <inertial>
@@ -34,24 +23,24 @@
                iyy="0.00000001"
                iyz="0.00"
-               izz="0.00000001"/> <!-- ${base_mass_kg/12*(base_x_m**2 + base_z_m**2)} -->
+               izz="0.00000001"/>
     </inertial>
-  </link>
+  </link> -->
   <link name="base_link">
     <visual>
-      <origin rpy="0 ${3.1415/2} 0" />
+      <!-- <origin rpy="0 ${3.1415/2} 0" /> -->
       <geometry>
-        <cylinder radius="0.01" length="0.05" />
+        <box size="0.05 0.05 0.01" />
       </geometry>
     </visual>
     <collision name="base_collision">
-      <origin rpy="0 ${3.1415/2} 0" />
+      <!-- <origin rpy="0 ${3.1415/2} 0" /> -->
       <geometry>
-        <cylinder radius="0.01" length="0.05" />
+        <box size="0.05 0.05 0.01" />
       </geometry>
       <surface>
         <friction>
           <ode>
-            <mu>0.6</mu>
-            <mu2>0.6</mu2>
+            <mu>200.0</mu>
+            <mu2>200.0</mu2>
           </ode>
         </friction>
@@ -60,10 +49,10 @@
     <inertial>
       <mass value="${base_mass_kg}"/>
-      <inertia ixx="0.00000001"
+      <inertia ixx="10"
                ixy="0.00"
                ixz="0.00"
-               iyy="0.00000001"
+               iyy="10"
                iyz="0.00"
-               izz="0.00000001"/> <!-- ${base_mass_kg/12*(base_x_m**2 + base_z_m**2)} -->
+               izz="10"/> <!-- ${base_mass_kg/12*(base_x_m**2 + base_z_m**2)} -->
     </inertial>
     <!-- <sensor name="base_contact" type="contact">
@@ -74,5 +63,5 @@
     </sensor> -->
   </link>
-  <joint name="world_base_theta" type="continuous">
+  <!-- <joint name="world_base_theta" type="continuous">
     <parent link="world" />
     <child link="base0" />
@@ -80,7 +69,7 @@
     <origin rpy="0 0 0" xyz="0 0 0"/>
     <limit effort="1000" velocity="1000" />
-  </joint>
-  <joint name="world_base_z" type="prismatic">
-    <parent link="base0" />
+  </joint> -->
+  <!-- <joint name="world_base_z" type="prismatic">
+    <parent link="world" />
     <child link="base1" />
     <axis xyz="0 0 1" />
@@ -94,5 +83,5 @@
     <origin rpy="0 0 0" xyz="0 0 0"/>
     <limit lower="-1000" upper="1000" effort="1000" velocity="1000" />
-  </joint>
+  </joint> -->
   <xacro:arm length="${arm_length_m}"
              width="${arm_width_m}"

Commit message: Succesfully set friction on arm link
moved the friction tag so it's specified after the
arm is specified

File: urdf/arm.xacro (robot description, xacro)
@@ -10,10 +10,10 @@
       </geometry>
     </visual>
-    <!--collision>
+    <collision>
       <origin rpy="0 0 0" xyz="0 0 ${length/2}"/>
       <geometry>
         <box size="${width} ${width} ${length}"/>
       </geometry>
-    </collision-->
+    </collision>
     <inertial>
       <origin rpy="0 0 0" xyz="0 0 ${length/2}"/>

File: urdf/pendulum.xacro (robot description, xacro)
@@ -26,10 +26,4 @@
     </inertial>
   </link> -->
-  <gazebo reference="base_link">
-    <mu1>0.2</mu1>
-    <mu2>0.2</mu2>
-    <kp>300</kp>
-    <material>Gazebo/Red</material>
-  </gazebo>
   <link name="base_link">
     <visual>
@@ -108,4 +102,10 @@
     <origin rpy="0 0 0" xyz="0 0 ${2 * base_z_m - 1}"/>
   </joint> -->
+  <gazebo reference="arm_link">
+    <mu1>0.2</mu1>
+    <mu2>0.2</mu2>
+    <kp>300</kp>
+    <material>Gazebo/Red</material>
+  </gazebo>
   <!-- Add ROS plugin so we can interact with our robot -->
   <gazebo>

Commit message: Merge with remote

File: urdf/arm.xacro (robot description, xacro)
@@ -10,10 +10,10 @@
       </geometry>
     </visual>
-    <!--collision>
+    <!-- <collision>
       <origin rpy="0 0 0" xyz="0 0 ${length/2}"/>
       <geometry>
         <box size="${width} ${width} ${length}"/>
       </geometry>
-    </collision-->
+    </collision> -->
     <inertial>
       <origin rpy="0 0 0" xyz="0 0 ${length/2}"/>
@@ -30,5 +30,4 @@
     <inertial>
       <origin rpy="0 0 0" xyz="0 0 0"/>
-      <!-- holds the mass of the solenoid, DSTL-0829-12 -->
       <mass value="0.001"/>
       <inertia ixx="0.0000001"
@@ -53,6 +52,6 @@
   </link> -->
   <joint name="base_free_theta" type="continuous">
-    <parent link="base_link" />
-    <child link="arm0_link" />
+    <parent link="arm0_link" />
+    <child link="arm_link" />
     <axis xyz="1 0 0" />
     <origin rpy="0 0 0" xyz="0 0 0"/>
@@ -61,6 +60,6 @@
   <joint name="arm_spring" type="prismatic">
     <axis xyz="0 0 1" />
-    <parent link="arm0_link" />
-    <child link="arm_link" />
+    <parent link="base_link" />
+    <child link="arm0_link" />
     <origin rpy="0 0 0" xyz="0 0 0"/>
     <!-- <dynamics friction="0" damping="50" /> --> <!-- implement dynamics using the PID controller (D = damping) -->

File: urdf/pendulum.xacro (robot description, xacro)
@@ -30,5 +30,4 @@
     <mu2>200</mu2>
     <!-- <kp>30000</kp> -->
-    <material>Gazebo/Red</material>
   </gazebo>
   <link name="base_link">

Commit message: Try to make a servo piston using position joint
ODE doesn't like D=1.4. Go figure. Will try to do this softer with a
custom effort-based controller.

Also, oops, forgot all this time to include `util.cpp`

File: urdf/arm.xacro (robot description, xacro)
@@ -88,13 +88,4 @@
     </joint>
   </transmission>
-  <transmission name="$arm_prism_transmission">
-    <type>transmission_interface/SimpleTransmission</type>
-    <actuator name="$arm_prism_motor">
-      <mechanicalReduction>1</mechanicalReduction>
-    </actuator>
-    <joint name="arm_prism">
-      <hardwareInterface>hardware_interface/EffortJointInterface</hardwareInterface>
-    </joint>
-  </transmission>
 </xacro:macro>
 </robot>

File: urdf/flywheel.xacro (robot description, xacro)
@@ -23,5 +23,15 @@
       </inertial>
     </link>
+    <gazebo reference="arm2_link">
+      <!-- must come before the link definition (major ???) -->
+      <material>Gazebo/Blue</material>
+    </gazebo>
     <link name="arm2_link">
+      <visual>
+        <origin rpy="0 0 0" xyz="0.01 0 0.0127"/>
+        <geometry>
+          <cylinder length="0.0254" radius="0.00254"/>
+        </geometry>
+      </visual>
       <inertial>
         <origin rpy="0 0 0" xyz="0 0 0"/>
@@ -35,24 +45,90 @@
       </inertial>
     </link>
-    <joint name="arm_prism" type="prismatic">
+    <gazebo reference="arm3_link">
+      <!-- must come before the link definition (major ???) -->
+      <material>Gazebo/Blue</material>
+    </gazebo>
+    <link name="arm3_link">
+      <visual>
+        <origin rpy="0 ${3.1415/2} 0" xyz="0.01 0 0.0127"/>
+        <geometry>
+          <cylinder length="0.002" radius="0.0127"/>
+        </geometry>
+      </visual>
+      <inertial>
+        <origin rpy="0 0 0" xyz="0 0 0.0127"/>
+        <mass value="0.001"/>
+        <inertia ixx="0.000001"
+                 ixy="0.00"
+                 ixz="0.00"
+                 iyy="0.000001"
+                 iyz="0.00"
+                 izz="0.000001"/>
+      </inertial>
+    </link>
+    <link name="arm4_link">
+      <inertial>
+        <origin rpy="0 0 0" xyz="0 0 0"/>
+        <mass value="0.001"/>
+        <inertia ixx="0.000001"
+                 ixy="0.00"
+                 ixz="0.00"
+                 iyy="0.000001"
+                 iyz="0.00"
+                 izz="0.000001"/>
+      </inertial>
+    </link>
+    <!-- <joint name="arm_prism" type="prismatic">
       <axis xyz="0 0 1" />
       <parent link="arm_link" />
       <child link="arm2_link" />
       <origin rpy="0 0 0" xyz="0 0 0"/>
-      <!-- <dynamics friction="0" damping="50" /> --> <!-- implement dynamics using the PID controller (D = damping) -->
       <limit lower="0.006" upper="0.013" effort="1000" velocity="1000" />
+    </joint> -->
+    <joint name="arm_piston_base" type="continuous">
+      <axis xyz="1 0 0" />
+      <parent link="arm_link" />
+      <child link="arm2_link" />
+      <origin rpy="0 0 0" xyz="0 0 ${arm_length}"/>
     </joint>
+    <joint name="arm_piston_top" type="continuous">
+      <axis xyz="1 0 0" />
+      <parent link="arm2_link" />
+      <child link="arm3_link" />
+      <origin rpy="0 0 0" xyz="0 0 0.0254"/>
+    </joint>
+    <joint name="arm_piston_driver" type="revolute">
+      <axis xyz="1 0 0" />
+      <parent link="arm3_link" />
+      <child link="arm4_link" />
+      <origin rpy="0 0 0" xyz="0 0 0.0127"/>
+      <limit lower="${-3.1415*7/8}" upper="${-3.1415*1/8}" effort="1000" velocity="1000" />
+    </joint>
+    <gazebo>
+      <joint name="arm_piston_align" type="prismatic">
+        <axis>
+          <xyz>0 0 1</xyz>
+          <limit>
+            <lower>-1</lower>
+            <upper>1</upper>
+          </limit>
+        </axis>
+        <parent>arm_link</parent>
+        <child>arm4_link</child>
+        <pose>0 0 0.00127 0 0 0</pose>
+      </joint>
+    </gazebo>
     <joint name="arm_to_flywheel" type="continuous">
       <axis xyz="0 0 1"/>
-      <parent link="arm2_link"/>
+      <parent link="arm4_link"/>
       <child link="flywheel_link"/>
-      <origin rpy="0 ${3.1415/2} 0" xyz="0 0 ${arm_length}"/> <!-- ${offset} -->
+      <origin rpy="0 ${3.1415/2} 0" xyz="0 0 ${radius}"/> <!-- ${offset} -->
     </joint>
-    <transmission name="$arm_prism_transmission">
+    <transmission name="$arm_piston_transmission">
       <type>transmission_interface/SimpleTransmission</type>
-      <actuator name="$arm_prism_motor">
+      <actuator name="$arm_piston_motor">
         <mechanicalReduction>1</mechanicalReduction>
       </actuator>
-      <joint name="arm_prism">
+      <joint name="arm_piston_driver">
         <hardwareInterface>hardware_interface/EffortJointInterface</hardwareInterface>
       </joint>
