Commit message: Use CLion's automatic code refactoring
Refactoring function will help to make code consistent.
Currently just using the default code style with indent=2

File: urdf/pendulum.xacro (robot description, xacro)
@@ -1,122 +1,122 @@
 <?xml version="1.0"?>
 <robot xmlns:xacro="http://www.ros.org/wiki/xacro" name="pendulum">
-  <xacro:include filename="$(find pendulum)/urdf/arm.xacro" />
-  <xacro:include filename="$(find pendulum)/urdf/flywheel.xacro" />
-  <xacro:property name="base_mass_kg" value="0.001" />
-  <xacro:property name="base_x_m" value=".05" />
-  <xacro:property name="base_y_m" value=".05" />
-  <xacro:property name="base_z_m" value=".06" />
-  <xacro:property name="arm_linear_density_kg_m" value=".129" />
-  <xacro:property name="arm_length_m" value=".10" />
-  <xacro:property name="arm_width_m" value=".02" />
-  <xacro:property name="motor_mass_kg" value=".080" />
-  <xacro:property name="wheel_mass_kg" value=".037" />
-  <xacro:property name="solenoid_mass_kg" value="${.10206 * 2}" />
-  <xacro:property name="wheel_radius_m" value=".05" />
-  <xacro:property name="wheel_length_m" value=".02" />
-  <!-- <link name="world" />
-  <link name="base1">
-    <inertial>
-      <mass value="0.0001"/>
-      <inertia ixx="0.00000001"
-               ixy="0.00"
-               ixz="0.00"
-               iyy="0.00000001"
-               iyz="0.00"
-               izz="0.00000001"/>
-    </inertial>
-  </link> -->
-  <gazebo reference="base_link">
-    <mu1>200</mu1>
-    <mu2>200</mu2>
-    <!-- <kp>30000</kp> -->
-  </gazebo>
-  <link name="base_link">
-    <visual>
-      <!-- <origin rpy="0 ${3.1415/2} 0" /> -->
-      <geometry>
-        <box size="0.05 0.05 0.01" />
-      </geometry>
-    </visual>
-    <collision>
-      <!-- <origin rpy="0 ${3.1415/2} 0" /> -->
-      <geometry>
-        <box size="0.05 0.05 0.01" />
-      </geometry>
-      <!-- <surface>
-        <contact>
-          <ode>
-            <soft_cfm>0.3</soft_cfm>
-          </ode>
-        </contact>
-        <friction>
-          <ode>
-            <mu>200</mu>
-            <mu2>200</mu2>
-          </ode>
-        </friction>
-      </surface> -->
-    </collision>
-    <inertial>
-      <mass value="${base_mass_kg}"/>
-      <inertia ixx="10"
-               ixy="0.00"
-               ixz="0.00"
-               iyy="10"
-               iyz="0.00"
-               izz="10"/> <!-- ${base_mass_kg/12*(base_x_m**2 + base_z_m**2)} -->
-    </inertial>
-    <!-- <sensor name="base_contact" type="contact">
-      <contact>
-        <collision>base_collision</collision>
-      </contact>
-      <update_rate>60</update_rate>
-    </sensor> -->
-  </link>
-  <!-- <joint name="world_base_theta" type="continuous">
-    <parent link="world" />
-    <child link="base0" />
-    <axis xyz="1 0 0" />
-    <origin rpy="0 0 0" xyz="0 0 0"/>
-    <limit effort="1000" velocity="1000" />
-  </joint> -->
-  <!-- <joint name="world_base_z" type="prismatic">
-    <parent link="world" />
-    <child link="base1" />
-    <axis xyz="0 0 1" />
-    <origin rpy="0 0 0" xyz="0 0 0"/>
-    <limit lower="-1000" upper="1000" effort="1000" velocity="1000" />
-  </joint>
-  <joint name="world_base_y" type="prismatic">
-    <parent link="base1" />
-    <child link="base_link" />
-    <axis xyz="0 1 0" />
-    <origin rpy="0 0 0" xyz="0 0 0"/>
-    <limit lower="-1000" upper="1000" effort="1000" velocity="1000" />
-  </joint> -->
-  <xacro:arm length="${arm_length_m}"
-             width="${arm_width_m}"
-             linear_density="${arm_linear_density_kg_m}"/>
-  <xacro:flywheel length="${wheel_length_m}"
-                  radius="${wheel_radius_m}"
-                  mass="${wheel_mass_kg}"
-                  motor_mass="${motor_mass_kg}"
-                  arm_length="${arm_length_m}"
-                  solenoid_mass="${solenoid_mass_kg}" />
-                  <!-- offset="${arm_length_m}" -->
-  <!-- <joint name="fixed" type="fixed">
-    <parent link="world"/>
-    <child link="base_link"/>
-    <origin rpy="0 0 0" xyz="0 0 ${2 * base_z_m - 1}"/>
-  </joint> -->
-  <!-- Add ROS plugin so we can interact with our robot -->
-  <gazebo>
-    <plugin name="gazebo_ros_control" filename="libgazebo_ros_control.so">
-      <robotNamespace>/</robotNamespace>
-    </plugin>
-    <!-- <plugin name="v_naught" filename="libInitialVelocityPlugin.so">
-      <link>base_link</link>
-      <linear>0 4.0 0</linear>
-    </plugin> -->
-  </gazebo>
+    <xacro:include filename="$(find pendulum)/urdf/arm.xacro"/>
+    <xacro:include filename="$(find pendulum)/urdf/flywheel.xacro"/>
+    <xacro:property name="base_mass_kg" value="0.001"/>
+    <xacro:property name="base_x_m" value=".05"/>
+    <xacro:property name="base_y_m" value=".05"/>
+    <xacro:property name="base_z_m" value=".06"/>
+    <xacro:property name="arm_linear_density_kg_m" value=".129"/>
+    <xacro:property name="arm_length_m" value=".10"/>
+    <xacro:property name="arm_width_m" value=".02"/>
+    <xacro:property name="motor_mass_kg" value=".080"/>
+    <xacro:property name="wheel_mass_kg" value=".037"/>
+    <xacro:property name="solenoid_mass_kg" value="${.10206 * 2}"/>
+    <xacro:property name="wheel_radius_m" value=".05"/>
+    <xacro:property name="wheel_length_m" value=".02"/>
+    <!-- <link name="world" />
+    <link name="base1">
+      <inertial>
+        <mass value="0.0001"/>
+        <inertia ixx="0.00000001"
+                 ixy="0.00"
+                 ixz="0.00"
+                 iyy="0.00000001"
+                 iyz="0.00"
+                 izz="0.00000001"/>
+      </inertial>
+    </link> -->
+    <gazebo reference="base_link">
+        <mu1>200</mu1>
+        <mu2>200</mu2>
+        <!-- <kp>30000</kp> -->
+    </gazebo>
+    <link name="base_link">
+        <visual>
+            <!-- <origin rpy="0 ${3.1415/2} 0" /> -->
+            <geometry>
+                <box size="0.05 0.05 0.01"/>
+            </geometry>
+        </visual>
+        <collision>
+            <!-- <origin rpy="0 ${3.1415/2} 0" /> -->
+            <geometry>
+                <box size="0.05 0.05 0.01"/>
+            </geometry>
+            <!-- <surface>
+              <contact>
+                <ode>
+                  <soft_cfm>0.3</soft_cfm>
+                </ode>
+              </contact>
+              <friction>
+                <ode>
+                  <mu>200</mu>
+                  <mu2>200</mu2>
+                </ode>
+              </friction>
+            </surface> -->
+        </collision>
+        <inertial>
+            <mass value="${base_mass_kg}"/>
+            <inertia ixx="10"
+                     ixy="0.00"
+                     ixz="0.00"
+                     iyy="10"
+                     iyz="0.00"
+                     izz="10"/> <!-- ${base_mass_kg/12*(base_x_m**2 + base_z_m**2)} -->
+        </inertial>
+        <!-- <sensor name="base_contact" type="contact">
+          <contact>
+            <collision>base_collision</collision>
+          </contact>
+          <update_rate>60</update_rate>
+        </sensor> -->
+    </link>
+    <!-- <joint name="world_base_theta" type="continuous">
+      <parent link="world" />
+      <child link="base0" />
+      <axis xyz="1 0 0" />
+      <origin rpy="0 0 0" xyz="0 0 0"/>
+      <limit effort="1000" velocity="1000" />
+    </joint> -->
+    <!-- <joint name="world_base_z" type="prismatic">
+      <parent link="world" />
+      <child link="base1" />
+      <axis xyz="0 0 1" />
+      <origin rpy="0 0 0" xyz="0 0 0"/>
+      <limit lower="-1000" upper="1000" effort="1000" velocity="1000" />
+    </joint>
+    <joint name="world_base_y" type="prismatic">
+      <parent link="base1" />
+      <child link="base_link" />
+      <axis xyz="0 1 0" />
+      <origin rpy="0 0 0" xyz="0 0 0"/>
+      <limit lower="-1000" upper="1000" effort="1000" velocity="1000" />
+    </joint> -->
+    <xacro:arm length="${arm_length_m}"
+               width="${arm_width_m}"
+               linear_density="${arm_linear_density_kg_m}"/>
+    <xacro:flywheel length="${wheel_length_m}"
+                    radius="${wheel_radius_m}"
+                    mass="${wheel_mass_kg}"
+                    motor_mass="${motor_mass_kg}"
+                    arm_length="${arm_length_m}"
+                    solenoid_mass="${solenoid_mass_kg}"/>
+    <!-- offset="${arm_length_m}" -->
+    <!-- <joint name="fixed" type="fixed">
+      <parent link="world"/>
+      <child link="base_link"/>
+      <origin rpy="0 0 0" xyz="0 0 ${2 * base_z_m - 1}"/>
+    </joint> -->
+    <!-- Add ROS plugin so we can interact with our robot -->
+    <gazebo>
+        <plugin name="gazebo_ros_control" filename="libgazebo_ros_control.so">
+            <robotNamespace>/</robotNamespace>
+        </plugin>
+        <!-- <plugin name="v_naught" filename="libInitialVelocityPlugin.so">
+          <link>base_link</link>
+          <linear>0 4.0 0</linear>
+        </plugin> -->
+    </gazebo>
 </robot>

File: urdf/tracker.xacro (robot description, xacro)
@@ -1,44 +1,44 @@
 <?xml version="1.0"?>
 <robot xmlns:xacro="http://www.ros.org/wiki/xacro" name="tracker">
-  <link name="world" />
-  <!-- <gazebo>
-  	<gravity>false</gravity>
-  </gazebo> -->
-  <gazebo reference="tracking_dot">
-  	<!-- must come before the link definition (major ???) -->
-  	<material>Gazebo/Red</material>
-  </gazebo>
-  <link name="tracking_dot">
-  	<visual>
-      <origin xyz="0 0 0.015" />
-      <geometry>
-        <box size="0.03 0.03 0.03" />
-      </geometry>
-      <material name="red">
-      	<color rgba="1.0 0 0 1.0" />
-      </material>
-    </visual>
-  	<!-- <collision>
-      <origin xyz="0 0 0.015" />
-      <geometry>
-        <box size="0.03 0.03 0.03" />
-      </geometry>
-    </collision> -->
-    <inertial>
-      <mass value="0.001"/>
-      <inertia ixx="1"
-               ixy="0.00"
-               ixz="0.00"
-               iyy="1"
-               iyz="0.00"
-               izz="1"/> <!-- ${base_mass_kg/12*(base_x_m**2 + base_z_m**2)} -->
-    </inertial>
-  </link>
-  <joint name="tracker" type="prismatic">
-    <axis xyz="0 1 0" />
-  	<parent link="world" />
-  	<child link="tracking_dot" />
-    <origin rpy="0 0 0" xyz="0 0 0"/>
-    <limit lower="-100" upper="100" effort="1000" velocity="1000" />
-  </joint>
+    <link name="world"/>
+    <!-- <gazebo>
+        <gravity>false</gravity>
+    </gazebo> -->
+    <gazebo reference="tracking_dot">
+        <!-- must come before the link definition (major ???) -->
+        <material>Gazebo/Red</material>
+    </gazebo>
+    <link name="tracking_dot">
+        <visual>
+            <origin xyz="0 0 0.015"/>
+            <geometry>
+                <box size="0.03 0.03 0.03"/>
+            </geometry>
+            <material name="red">
+                <color rgba="1.0 0 0 1.0"/>
+            </material>
+        </visual>
+        <!-- <collision>
+        <origin xyz="0 0 0.015" />
+        <geometry>
+          <box size="0.03 0.03 0.03" />
+        </geometry>
+      </collision> -->
+        <inertial>
+            <mass value="0.001"/>
+            <inertia ixx="1"
+                     ixy="0.00"
+                     ixz="0.00"
+                     iyy="1"
+                     iyz="0.00"
+                     izz="1"/> <!-- ${base_mass_kg/12*(base_x_m**2 + base_z_m**2)} -->
+        </inertial>
+    </link>
+    <joint name="tracker" type="prismatic">
+        <axis xyz="0 1 0"/>
+        <parent link="world"/>
+        <child link="tracking_dot"/>
+        <origin rpy="0 0 0" xyz="0 0 0"/>
+        <limit lower="-100" upper="100" effort="1000" velocity="1000"/>
+    </joint>
 </robot>

Commit message: flip the order of joints to match real world robot

File: urdf/arm.xacro (robot description, xacro)
@@ -52,6 +52,6 @@
         </link> -->
         <joint name="base_free_theta" type="continuous">
-            <parent link="arm0_link"/>
-            <child link="arm_link"/>
+            <parent link="base_link"/>
+            <child link="arm0_link"/>
             <axis xyz="1 0 0"/>
             <origin rpy="0 0 0" xyz="0 0 0"/>
@@ -59,7 +59,7 @@
         </joint>
         <joint name="arm_spring" type="prismatic">
+            <parent link="arm0_link"/>
+            <child link="arm_link"/>
             <axis xyz="0 0 1"/>
-            <parent link="base_link"/>
-            <child link="arm0_link"/>
             <origin rpy="0 0 0" xyz="0 0 0"/>
             <!-- <dynamics friction="0" damping="50" /> --> <!-- implement dynamics using the PID controller (D = damping) -->

Commit message: Make test setup for validating Python sim
Anchor the arm spring joint to the world, set the initial position of the
spring, all for testing the Python sim accuracy via comparing final energy.

File: urdf/arm.xacro (robot description, xacro)
@@ -18,5 +18,5 @@
             <inertial>
                 <origin rpy="0 0 0" xyz="0 0 ${length/2}"/>
-                <mass value="${linear_density * length}"/>
+                <mass value="0.0001" /> <!-- ${linear_density * length}"/> -->
                 <inertia ixx="${mass/12*(width**2 + width**2)}"
                          ixy="0.00"
@@ -27,5 +27,5 @@
             </inertial>
         </link>
-        <link name="arm0_link">
+        <!-- <link name="arm0_link">
             <inertial>
                 <origin rpy="0 0 0" xyz="0 0 0"/>
@@ -39,5 +39,5 @@
             </inertial>
         </link>
-        <!-- <link name="arm1_link">
+        <link name="arm1_link">
           <inertial>
             <origin rpy="0 0 0" xyz="0 0 0"/>
@@ -50,5 +50,5 @@
                      izz="10"/>
           </inertial>
-        </link> -->
+        </link>
         <joint name="base_free_theta" type="continuous">
             <parent link="base_link"/>
@@ -57,7 +57,7 @@
             <origin rpy="0 0 0" xyz="0 0 0"/>
             <limit effort="1000" velocity="1000"/>
-        </joint>
+        </joint> -->
         <joint name="arm_spring" type="prismatic">
-            <parent link="arm0_link"/>
+            <parent link="world"/>
             <child link="arm_link"/>
             <axis xyz="0 0 1"/>

File: urdf/pendulum.xacro (robot description, xacro)
@@ -12,87 +12,8 @@
     <xacro:property name="motor_mass_kg" value=".080"/>
     <xacro:property name="wheel_mass_kg" value=".037"/>
-    <xacro:property name="solenoid_mass_kg" value="${.10206 * 2}"/>
+    <xacro:property name="solenoid_mass_kg" value="${0.350 - motor_mass_kg - wheel_mass_kg}"/> <!-- hack it to get 350g -->
     <xacro:property name="wheel_radius_m" value=".05"/>
     <xacro:property name="wheel_length_m" value=".02"/>
-    <!-- <link name="world" />
-    <link name="base1">
-      <inertial>
-        <mass value="0.0001"/>
-        <inertia ixx="0.00000001"
-                 ixy="0.00"
-                 ixz="0.00"
-                 iyy="0.00000001"
-                 iyz="0.00"
-                 izz="0.00000001"/>
-      </inertial>
-    </link> -->
-    <gazebo reference="base_link">
-        <mu1>200</mu1>
-        <mu2>200</mu2>
-        <!-- <kp>30000</kp> -->
-    </gazebo>
-    <link name="base_link">
-        <visual>
-            <!-- <origin rpy="0 ${3.1415/2} 0" /> -->
-            <geometry>
-                <box size="0.05 0.05 0.01"/>
-            </geometry>
-        </visual>
-        <collision>
-            <!-- <origin rpy="0 ${3.1415/2} 0" /> -->
-            <geometry>
-                <box size="0.05 0.05 0.01"/>
-            </geometry>
-            <!-- <surface>
-              <contact>
-                <ode>
-                  <soft_cfm>0.3</soft_cfm>
-                </ode>
-              </contact>
-              <friction>
-                <ode>
-                  <mu>200</mu>
-                  <mu2>200</mu2>
-                </ode>
-              </friction>
-            </surface> -->
-        </collision>
-        <inertial>
-            <mass value="${base_mass_kg}"/>
-            <inertia ixx="10"
-                     ixy="0.00"
-                     ixz="0.00"
-                     iyy="10"
-                     iyz="0.00"
-                     izz="10"/> <!-- ${base_mass_kg/12*(base_x_m**2 + base_z_m**2)} -->
-        </inertial>
-        <!-- <sensor name="base_contact" type="contact">
-          <contact>
-            <collision>base_collision</collision>
-          </contact>
-          <update_rate>60</update_rate>
-        </sensor> -->
-    </link>
-    <!-- <joint name="world_base_theta" type="continuous">
-      <parent link="world" />
-      <child link="base0" />
-      <axis xyz="1 0 0" />
-      <origin rpy="0 0 0" xyz="0 0 0"/>
-      <limit effort="1000" velocity="1000" />
-    </joint> -->
-    <!-- <joint name="world_base_z" type="prismatic">
-      <parent link="world" />
-      <child link="base1" />
-      <axis xyz="0 0 1" />
-      <origin rpy="0 0 0" xyz="0 0 0"/>
-      <limit lower="-1000" upper="1000" effort="1000" velocity="1000" />
-    </joint>
-    <joint name="world_base_y" type="prismatic">
-      <parent link="base1" />
-      <child link="base_link" />
-      <axis xyz="0 1 0" />
-      <origin rpy="0 0 0" xyz="0 0 0"/>
-      <limit lower="-1000" upper="1000" effort="1000" velocity="1000" />
-    </joint> -->
+    <link name="world" />
     <xacro:arm length="${arm_length_m}"
                width="${arm_width_m}"

Commit message: increase mass values to help numerical stability
Seems like setting link mass near zero is the cause for velocity
instability. I remembered in Robosoccer we ran into similar issue
The velocity is no longer jerky, we may try to increase step size
to speed up simulation

File: urdf/arm.xacro (robot description, xacro)
@@ -10,13 +10,7 @@
                 </geometry>
             </visual>
-            <!-- <collision>
-              <origin rpy="0 0 0" xyz="0 0 ${length/2}"/>
-              <geometry>
-                <box size="${width} ${width} ${length}"/>
-              </geometry>
-            </collision> -->
             <inertial>
                 <origin rpy="0 0 0" xyz="0 0 ${length/2}"/>
-                <mass value="0.0001" /> <!-- ${linear_density * length}"/> -->
+                <mass value="0.001" /> <!-- ${linear_density * length}"/> -->
                 <inertia ixx="${mass/12*(width**2 + width**2)}"
                          ixy="0.00"

File: urdf/flywheel.xacro (robot description, xacro)
@@ -9,9 +9,4 @@
                 </geometry>
             </visual>
-            <!-- <collision>
-              <geometry>
-                <cylinder length="${length}" radius="${radius}"/>
-              </geometry>
-            </collision> -->
             <inertial>
                 <mass value="${mass + motor_mass + solenoid_mass}"/>
@@ -60,5 +55,5 @@
                 <origin rpy="0 0 0" xyz="0 -0.01 0.0"/>
                 <mass value="0.001"/>
-                <inertia ixx="0.000001"
+                <inertia ixx="0.001"
                          ixy="0.00"
                          ixz="0.00"
@@ -72,5 +67,5 @@
                 <origin rpy="0 0 0" xyz="0 0 0"/>
                 <mass value="0.001"/>
-                <inertia ixx="0.000001"
+                <inertia ixx="0.001"
                          ixy="0.00"
                          ixz="0.00"
