Commit message: clean up urdf files

File: urdf/arm.xacro (robot description, xacro)
@@ -7,13 +7,7 @@
                 <origin rpy="0 0 0" xyz="0 0 ${length/2}"/>
                 <geometry>
-                    <box size="${width} ${width} ${length}"/>
+                    <cylinder radius="${width/2}" length="${length}"/>
                 </geometry>
             </visual>
-            <!-- <collision>
-              <origin rpy="0 0 0" xyz="0 0 ${length/2}"/>
-              <geometry>
-                <box size="${width} ${width} ${length}"/>
-              </geometry>
-            </collision> -->
             <inertial>
                 <origin rpy="0 0 0" xyz="0 0 ${length/2}"/>
@@ -39,16 +33,4 @@
             </inertial>
         </link>
-        <!-- <link name="arm1_link">
-          <inertial>
-            <origin rpy="0 0 0" xyz="0 0 0"/>
-            <mass value="0.001"/>
-            <inertia ixx="0"
-                     ixy="0.00"
-                     ixz="0.00"
-                     iyy="10"
-                     iyz="0.00"
-                     izz="10"/>
-          </inertial>
-        </link> -->
         <joint name="base_free_theta" type="continuous">
             <parent link="base_link"/>
@@ -66,17 +48,4 @@
             <limit lower="-1" upper="0" effort="1000" velocity="1000"/>
         </joint>
-        <!-- <joint name="arm_fix" type="fixed">
-          <parent link="arm1_link" />
-          <child link="arm2_link" />
-        </joint> -->
-        <!-- <transmission name="$arm_transmission">
-          <type>transmission_interface/SimpleTransmission</type>
-          <actuator name="$arm_motor">
-            <mechanicalReduction>1</mechanicalReduction>
-          </actuator>
-          <joint name="base_to_arm">
-            <hardwareInterface>hardware_interface/EffortJointInterface</hardwareInterface>
-          </joint>
-        </transmission> -->
         <transmission name="$arm_spring_transmission">
             <type>transmission_interface/SimpleTransmission</type>

File: urdf/flywheel.xacro (robot description, xacro)
@@ -9,9 +9,4 @@
                 </geometry>
             </visual>
-            <!-- <collision>
-              <geometry>
-                <cylinder length="${length}" radius="${radius}"/>
-              </geometry>
-            </collision> -->
             <inertial>
                 <mass value="${mass + motor_mass + solenoid_mass}"/>
@@ -80,23 +75,4 @@
             </inertial>
         </link>
-        <!-- <link name="arm5_link">
-          <inertial>
-            <origin rpy="0 0 0" xyz="0 0 0"/>
-            <mass value="0.001"/>
-            <inertia ixx="0.000001"
-                     ixy="0.00"
-                     ixz="0.00"
-                     iyy="0.000001"
-                     iyz="0.00"
-                     izz="0.000001"/>
-          </inertial>
-        </link> -->
-        <!-- <joint name="arm_prism" type="prismatic">
-          <axis xyz="0 0 1" />
-          <parent link="arm_link" />
-          <child link="arm2_link" />
-          <origin rpy="0 0 0" xyz="0 0 0"/>
-          <limit lower="0.006" upper="0.013" effort="1000" velocity="1000" />
-        </joint> -->
         <joint name="arm_piston_base" type="continuous">
             <axis xyz="1 0 0"/>

File: urdf/pendulum.xacro (robot description, xacro)
@@ -15,46 +15,18 @@
     <xacro:property name="wheel_radius_m" value=".05"/>
     <xacro:property name="wheel_length_m" value=".02"/>
-    <!-- <link name="world" />
-    <link name="base1">
-      <inertial>
-        <mass value="0.0001"/>
-        <inertia ixx="0.00000001"
-                 ixy="0.00"
-                 ixz="0.00"
-                 iyy="0.00000001"
-                 iyz="0.00"
-                 izz="0.00000001"/>
-      </inertial>
-    </link> -->
     <gazebo reference="base_link">
         <mu1>200</mu1>
         <mu2>200</mu2>
-        <!-- <kp>30000</kp> -->
     </gazebo>
     <link name="base_link">
         <visual>
-            <!-- <origin rpy="0 ${3.1415/2} 0" /> -->
             <geometry>
-                <box size="0.05 0.05 0.01"/>
+                <sphere radius="0.01"/>
             </geometry>
         </visual>
         <collision>
-            <!-- <origin rpy="0 ${3.1415/2} 0" /> -->
             <geometry>
-                <box size="0.05 0.05 0.01"/>
+                <sphere radius="0.01"/>
             </geometry>
-            <!-- <surface>
-              <contact>
-                <ode>
-                  <soft_cfm>0.3</soft_cfm>
-                </ode>
-              </contact>
-              <friction>
-                <ode>
-                  <mu>200</mu>
-                  <mu2>200</mu2>
-                </ode>
-              </friction>
-            </surface> -->
         </collision>
         <inertial>
@@ -67,32 +39,5 @@
                      izz="10"/> <!-- ${base_mass_kg/12*(base_x_m**2 + base_z_m**2)} -->
         </inertial>
-        <!-- <sensor name="base_contact" type="contact">
-          <contact>
-            <collision>base_collision</collision>
-          </contact>
-          <update_rate>60</update_rate>
-        </sensor> -->
     </link>
-    <!-- <joint name="world_base_theta" type="continuous">
-      <parent link="world" />
-      <child link="base0" />
-      <axis xyz="1 0 0" />
-      <origin rpy="0 0 0" xyz="0 0 0"/>
-      <limit effort="1000" velocity="1000" />
-    </joint> -->
-    <!-- <joint name="world_base_z" type="prismatic">
-      <parent link="world" />
-      <child link="base1" />
-      <axis xyz="0 0 1" />
-      <origin rpy="0 0 0" xyz="0 0 0"/>
-      <limit lower="-1000" upper="1000" effort="1000" velocity="1000" />
-    </joint>
-    <joint name="world_base_y" type="prismatic">
-      <parent link="base1" />
-      <child link="base_link" />
-      <axis xyz="0 1 0" />
-      <origin rpy="0 0 0" xyz="0 0 0"/>
-      <limit lower="-1000" upper="1000" effort="1000" velocity="1000" />
-    </joint> -->
     <xacro:arm length="${arm_length_m}"
                width="${arm_width_m}"
@@ -104,10 +49,4 @@
                     arm_length="${arm_length_m}"
                     solenoid_mass="${solenoid_mass_kg}"/>
-    <!-- offset="${arm_length_m}" -->
-    <!-- <joint name="fixed" type="fixed">
-      <parent link="world"/>
-      <child link="base_link"/>
-      <origin rpy="0 0 0" xyz="0 0 ${2 * base_z_m - 1}"/>
-    </joint> -->
     <!-- Add ROS plugin so we can interact with our robot -->
     <gazebo>
@@ -115,8 +54,4 @@
             <robotNamespace>/</robotNamespace>
         </plugin>
-        <!-- <plugin name="v_naught" filename="libInitialVelocityPlugin.so">
-          <link>base_link</link>
-          <linear>0 4.0 0</linear>
-        </plugin> -->
     </gazebo>
 </robot>

Commit message: remove free joint at the leg

File: urdf/arm.xacro (robot description, xacro)
@@ -21,25 +21,6 @@
             </inertial>
         </link>
-        <link name="arm0_link">
-            <inertial>
-                <origin rpy="0 0 0" xyz="0 0 0"/>
-                <mass value="0.001"/>
-                <inertia ixx="0.0000001"
-                         ixy="0.00"
-                         ixz="0.00"
-                         iyy="0.0000001"
-                         iyz="0.00"
-                         izz="0.0000001"/>
-            </inertial>
-        </link>
-        <joint name="base_free_theta" type="continuous">
+        <joint name="arm_spring" type="prismatic">
             <parent link="base_link"/>
-            <child link="arm0_link"/>
-            <axis xyz="1 0 0"/>
-            <origin rpy="0 0 0" xyz="0 0 0"/>
-            <limit effort="1000" velocity="1000"/>
-        </joint>
-        <joint name="arm_spring" type="prismatic">
-            <parent link="arm0_link"/>
             <child link="arm_link"/>
             <axis xyz="0 0 1"/>
