Commit message: rename joints in old model

File: pendulum/urdf/arm.xacro (robot description, xacro)
@@ -21,5 +21,5 @@
             </inertial>
         </link>
-        <joint name="arm_spring" type="prismatic">
+        <joint name="spring_joint" type="prismatic">
             <parent link="base_link"/>
             <child link="arm_link"/>
@@ -29,10 +29,10 @@
             <limit lower="-1" upper="0" effort="1000" velocity="1000"/>
         </joint>
-        <transmission name="$arm_spring_transmission">
+        <transmission name="$spring_joint_transmission">
             <type>transmission_interface/SimpleTransmission</type>
-            <actuator name="$arm_spring_motor">
+            <actuator name="$spring_joint_motor">
                 <mechanicalReduction>1</mechanicalReduction>
             </actuator>
-            <joint name="arm_spring">
+            <joint name="spring_joint">
                 <hardwareInterface>hardware_interface/EffortJointInterface</hardwareInterface>
             </joint>

File: pendulum/urdf/flywheel.xacro (robot description, xacro)
@@ -89,5 +89,5 @@
             <origin rpy="0 0 0" xyz="0 0 0.0254"/>
         </joint>
-        <joint name="arm_piston_driver" type="revolute">
+        <joint name="servo_joint" type="revolute">
             <axis xyz="1 0 0"/>
             <parent link="arm3_link"/>
@@ -110,5 +110,5 @@
             </joint>
         </gazebo>
-        <joint name="arm_to_flywheel" type="continuous">
+        <joint name="flywheel_joint" type="continuous">
             <axis xyz="0 0 1"/>
             <parent link="arm4_link"/>
@@ -121,5 +121,5 @@
                 <mechanicalReduction>1</mechanicalReduction>
             </actuator>
-            <joint name="arm_piston_driver">
+            <joint name="servo_joint">
                 <hardwareInterface>hardware_interface/EffortJointInterface</hardwareInterface>
             </joint>
@@ -130,5 +130,5 @@
                 <mechanicalReduction>1</mechanicalReduction>
             </actuator>
-            <joint name="arm_to_flywheel">
+            <joint name="flywheel_joint">
                 <hardwareInterface>hardware_interface/EffortJointInterface</hardwareInterface>
             </joint>

File: pendulum/urdf/pendulum.xacro (robot description, xacro)
@@ -3,5 +3,5 @@
     <xacro:include filename="$(find pendulum)/urdf/arm.xacro"/>
     <xacro:include filename="$(find pendulum)/urdf/flywheel.xacro"/>
-    <xacro:property name="base_mass_kg" value="0.001"/>
+    <xacro:property name="base_mass_kg" value="0.040"/>
     <xacro:property name="base_x_m" value=".05"/>
     <xacro:property name="base_y_m" value=".05"/>
@@ -51,7 +51,5 @@
     <!-- Add ROS plugin so we can interact with our robot -->
     <gazebo>
-        <plugin name="gazebo_ros_control" filename="libgazebo_ros_control.so">
-            <robotNamespace>/</robotNamespace>
-        </plugin>
+        <plugin name="gazebo_ros_control" filename="libgazebo_ros_control.so"/>
     </gazebo>
 </robot>
