Commit message: give spring wide limits, piston eyeball the limits

File: full_description/urdf/full.xacro (robot description, xacro)
@@ -240,5 +240,5 @@
   <child link="middle_v13_1"/>
   <axis xyz="-0.0 0.0 -1.0"/>
-  <limit effort="100" lower="0.0" upper="0.0" velocity="100"/>
+  <limit effort="100" lower="-0.0" upper="0.03" velocity="100"/>
 </joint>
 <joint name="spring_joint" type="prismatic">
@@ -247,5 +247,5 @@
   <child link="Leg_0_v2_1"/>
   <axis xyz="-0.0 0.0 -1.0"/>
-  <limit effort="100" lower="0.0" upper="0.0" velocity="100"/>
+  <limit effort="100" lower="-1.0" upper="1.0" velocity="100"/>
 </joint>
 <joint name="Rigid12" type="fixed">

Commit message: add spherical collision remove all other collisions

File: full_description/urdf/full.xacro (robot description, xacro)
@@ -17,10 +17,4 @@
     <material name="silver_default"/>
   </visual>
-  <collision>
-    <origin rpy="0 0 0" xyz="0 0 0"/>
-    <geometry>
-      <mesh filename="package://full_description/meshes/base_link.stl" scale="0.001 0.001 0.001"/>
-    </geometry>
-  </collision>
 </link>
 <link name="Savox_SV1270TG_v4_1">
@@ -37,10 +31,4 @@
     <material name="silver_default"/>
   </visual>
-  <collision>
-    <origin rpy="0 0 0" xyz="0.003047 -0.0202 -0.179703"/>
-    <geometry>
-      <mesh filename="package://full_description/meshes/Savox_SV1270TG_v4_1.stl" scale="0.001 0.001 0.001"/>
-    </geometry>
-  </collision>
 </link>
 <link name="battery_v2_1">
@@ -57,10 +45,4 @@
     <material name="silver_default"/>
   </visual>
-  <collision>
-    <origin rpy="0 0 0" xyz="0.002297 0.02945 -0.203703"/>
-    <geometry>
-      <mesh filename="package://full_description/meshes/battery_v2_1.stl" scale="0.001 0.001 0.001"/>
-    </geometry>
-  </collision>
 </link>
 <link name="_bldc_parts.d32996c5-cb5d-48d1-b36d-40a50d399b36_v5_1">
@@ -77,10 +59,4 @@
     <material name="silver_default"/>
   </visual>
-  <collision>
-    <origin rpy="0 0 0" xyz="-0.028253 -0.00705 -0.213703"/>
-    <geometry>
-      <mesh filename="package://full_description/meshes/_bldc_parts.d32996c5-cb5d-48d1-b36d-40a50d399b36_v5_1.stl" scale="0.001 0.001 0.001"/>
-    </geometry>
-  </collision>
 </link>
 <link name="Turnigy_Aerodrive_SK3_-_2836_v2_1">
@@ -97,10 +73,4 @@
     <material name="silver_default"/>
   </visual>
-  <collision>
-    <origin rpy="0 0 0" xyz="-0.033253 0.0012 -0.228977"/>
-    <geometry>
-      <mesh filename="package://full_description/meshes/Turnigy_Aerodrive_SK3_-_2836_v2_1.stl" scale="0.001 0.001 0.001"/>
-    </geometry>
-  </collision>
 </link>
 <link name="flywheel_v2_1">
@@ -117,10 +87,4 @@
     <material name="silver_default"/>
   </visual>
-  <collision>
-    <origin rpy="0 0 0" xyz="-0.070003 0.0012 -0.228977"/>
-    <geometry>
-      <mesh filename="package://full_description/meshes/flywheel_v2_1.stl" scale="0.001 0.001 0.001"/>
-    </geometry>
-  </collision>
 </link>
 <link name="9657K449_COMPRESSION_SPRING_v1_1">
@@ -137,10 +101,4 @@
     <material name="silver_default"/>
   </visual>
-  <collision>
-    <origin rpy="0 0 0" xyz="0.000147 -0.00055 -0.019803"/>
-    <geometry>
-      <mesh filename="package://full_description/meshes/9657K449_COMPRESSION_SPRING_v1_1.stl" scale="0.001 0.001 0.001"/>
-    </geometry>
-  </collision>
 </link>
 <link name="middle_v13_1">
@@ -157,10 +115,4 @@
     <material name="silver_default"/>
   </visual>
-  <collision>
-    <origin rpy="0 0 0" xyz="0.000147 -0.00055 -0.199703"/>
-    <geometry>
-      <mesh filename="package://full_description/meshes/middle_v13_1.stl" scale="0.001 0.001 0.001"/>
-    </geometry>
-  </collision>
 </link>
 <link name="Leg_0_v2_1">
@@ -177,10 +129,4 @@
     <material name="silver_default"/>
   </visual>
-  <collision>
-    <origin rpy="0 0 0" xyz="0.000147 -0.00055 -0.134603"/>
-    <geometry>
-      <mesh filename="package://full_description/meshes/Leg_0_v2_1.stl" scale="0.001 0.001 0.001"/>
-    </geometry>
-  </collision>
 </link>
 <link name="95495K673_POLYURETHANE_RUBBER_ADHESIVE-BACK_BUMPER_v1_1">
@@ -198,7 +144,7 @@
   </visual>
   <collision>
-    <origin rpy="0 0 0" xyz="0.000147 -0.00055 -0.011803"/>
-    <geometry>
-      <mesh filename="package://full_description/meshes/95495K673_POLYURETHANE_RUBBER_ADHESIVE-BACK_BUMPER_v1_1.stl" scale="0.001 0.001 0.001"/>
+    <origin rpy="0 0 0" xyz="0.0 0.0 0.0"/>
+    <geometry>
+      <sphere radius=".005"/>
     </geometry>
   </collision>

Commit message: add yaw flywheel to the model

File: full_description/urdf/full.xacro (robot description, xacro)
@@ -1,4 +1,5 @@
 <?xml version="1.0" ?>
 <robot name="full" xmlns:xacro="http://www.ros.org/wiki/xacro">
+<xacro:include filename="$(find pendulum)/urdf/imu.xacro"/>
 <xacro:include filename="$(find full_description)/urdf/materials.xacro" />
 <xacro:include filename="$(find full_description)/urdf/full.trans" />
@@ -18,4 +19,18 @@
   </visual>
 </link>
+<link name="yaw_flywheel">
+  <inertial>
+    <origin rpy="0 0 0" xyz="0 0 0"/>
+    <mass value="0.100"/>
+    <inertia ixx="1e-03" ixy="-0.0" ixz="-0.0" iyy="3.5e-05" iyz="-0.0" izz="3.5e-05"/>
+  </inertial>
+  <visual>
+    <origin rpy="0 0 0" xyz="0 0 0"/>
+    <geometry>
+      <box size=".05 .05 .01"/>
+    </geometry>
+    <material name="silver_default"/>
+  </visual>
+</link>
 <link name="Savox_SV1270TG_v4_1">
   <inertial>
@@ -77,6 +92,6 @@
   <inertial>
     <origin rpy="0 0 0" xyz="0.0014986943552602328 7.592667813915988e-15 -2.8213514774444448e-08"/>
-    <mass value="0.03660763962304266"/>
-    <inertia ixx="6.9e-05" ixy="-0.0" ixz="-0.0" iyy="3.5e-05" iyz="-0.0" izz="3.5e-05"/>
+    <mass value="0.100"/>
+    <inertia ixx="1e-03" ixy="-0.0" ixz="-0.0" iyy="3.5e-05" iyz="-0.0" izz="3.5e-05"/>
   </inertial>
   <visual>
@@ -169,4 +184,10 @@
   <parent link="_bldc_parts.d32996c5-cb5d-48d1-b36d-40a50d399b36_v5_1"/>
   <child link="Turnigy_Aerodrive_SK3_-_2836_v2_1"/>
+</joint>
+<joint name="yaw_flywheel_joint" type="continuous">
+  <origin rpy="0 0 0" xyz="0.0 0.0 0.25"/>
+  <parent link="base_link"/>
+  <child link="yaw_flywheel"/>
+  <axis xyz="0.0 0.0 1.0"/>
 </joint>
 <joint name="flywheel_joint" type="continuous">

Commit message: Add thrusters
Import `uuv_simulator`'s thruster plugins and start using them for force
generation. Fix inertias that were exported by Fusion2URDF as 0, which is
not handled well by ODE (seems to handle them like ~1kg*m^2)

File: full_description/urdf/full.xacro (robot description, xacro)
@@ -5,4 +5,7 @@
 <xacro:include filename="$(find full_description)/urdf/full.trans" />
 <xacro:include filename="$(find full_description)/urdf/full.gazebo" />
+<xacro:property name="COG_X" value="18.6E-3" />
+<xacro:property name="COG_Y" value="-0.717E-3" />
+<xacro:property name="COG_Z" value="202.078E-3" />
 <link name="base_link">
   <inertial>
@@ -107,5 +110,5 @@
     <origin rpy="0 0 0" xyz="0.000147 -0.00055 -0.019803"/>
     <mass value="0.0"/>
-    <inertia ixx="0.0" ixy="0.0" ixz="0.0" iyy="0.0" iyz="0.0" izz="0.0"/>
+    <inertia ixx="1.0E-7" ixy="0.0" ixz="0.0" iyy="1.0E-7" iyz="0.0" izz="1.0E-7"/>
   </inertial>
   <visual>
@@ -135,5 +138,5 @@
     <origin rpy="0 0 0" xyz="-4.2181849628047897e-07 -9.756626929979806e-15 0.028777697727251528"/>
     <mass value="0.04388165329610352"/>
-    <inertia ixx="0.000377" ixy="0.0" ixz="-0.0" iyy="0.000377" iyz="-0.0" izz="0.0"/>
+    <inertia ixx="0.000377" ixy="0.0" ixz="-0.0" iyy="0.000377" iyz="-0.0" izz="1E-7"/>
   </inertial>
   <visual>
@@ -149,5 +152,5 @@
     <origin rpy="0 0 0" xyz="0.000147 -0.00055 -0.011803"/>
     <mass value="0.0"/>
-    <inertia ixx="0.0" ixy="0.0" ixz="0.0" iyy="0.0" iyz="0.0" izz="0.0"/>
+    <inertia ixx="1.0E-7" ixy="0.0" ixz="0.0" iyy="1.0E-7" iyz="0.0" izz="1.0E-7"/>
   </inertial>
   <visual>
@@ -191,4 +194,33 @@
   <axis xyz="0.0 0.0 1.0"/>
 </joint>
+<xacro:macro name="thruster_link" params="id">
+  <link name="thruster_${id}">
+    <inertial>
+      <mass value="0.02" />
+      <origin xyz="0 0 0" rpy="0 0 0" />
+      <inertia ixx="5E-6" ixy="0" ixz="0"
+               iyy="2E-7" iyz="0"
+               izz="2E-7" />
+    </inertial>
+    <visual>
+      <origin rpy="0 1.57 0" xyz="0 0 0" />
+      <geometry>
+        <cylinder radius="14E-3" length="18E-3" />
+      </geometry>
+    </visual>
+  </link>
+</xacro:macro>
+<xacro:thruster_link id="0" />
+<xacro:thruster_link id="1" />
+<xacro:macro name="thruster_joint" params="id xyz">
+  <joint name="thruster_${id}_joint" type="continuous">
+    <origin rpy="0 0 0" xyz="${xyz}"/>
+    <axis xyz="1 0 0" />
+    <parent link="base_link" />
+    <child link="thruster_${id}" />
+  </joint>
+</xacro:macro>
+<xacro:thruster_joint xyz="${COG_X} ${COG_Y - 0.2} ${COG_Z}" id="0" />
+<xacro:thruster_joint xyz="${COG_X} ${COG_Y + 0.2} ${COG_Z}" id="1" />
 <joint name="flywheel_joint" type="continuous">
   <origin rpy="0 0 0" xyz="0.03675 0.0 0.0"/>
